File: AriG25Module.sch (KiCad schematic (older format))
At the start: 17 parts, among them J1 CON, U2 ARIA-G25

Commit message: Modified LAN9500A schematic.
Modified the schematic for the USB to Ethernet converter.
Parts:
- BT1: footprint (none) -> Battery_Holders:BatteryHolder_CoinCell_Keystone_3008
- C10, C11, C12, C13, C14, C15, C16, C17, C18, C7, C8, C9: footprint Capacitors_SMD:C_0603_HandSoldering -> Capacitors_SMD:C_0805_HandSoldering
- U2: footprint misc:ARIA-G25 -> (none)
Changed lines of the file:
@@
 F 0 "U2" H 4150 7050 60  0000 L BNB
 F 1 "ARIA-G25" H 4150 1250 40  0000 L TNN
-F 2 "misc:ARIA-G25" H 4150 1150 40  0001 L CNN
+F 2 "" H 4150 1150 40  0001 L CNN
 F 3 "" H 2200 5800 60  0001 C CNN
 F 4 "IC" H 4150 7150 40  0001 L BNN "Family"
@@
 F 0 "C10" H 2175 1750 50  0000 L CNN
 F 1 "1uF" V 2100 1450 50  0000 L CNN
-F 2 "Capacitors_SMD:C_0603_HandSoldering" H 2188 1500 50  0001 C CNN
+F 2 "Capacitors_SMD:C_0805_HandSoldering" H 2188 1500 50  0001 C CNN
 F 3 "" H 2150 1650 50  0000 C CNN
 	1    2150 1650
@@
 F 0 "C7" H 1975 1750 50  0000 L CNN
 F 1 "100nF" V 1900 1400 50  0000 L CNN
-F 2 "Capacitors_SMD:C_0603_HandSoldering" H 1988 1500 50  0001 C CNN
+F 2 "Capacitors_SMD:C_0805_HandSoldering" H 1988 1500 50  0001 C CNN
 F 3 "" H 1950 1650 50  0000 C CNN
 	1    1950 1650
@@
 F 0 "C17" H 3325 2050 50  0000 L CNN
 F 1 "100nF" V 3250 1650 50  0000 L CNN
-F 2 "Capacitors_SMD:C_0603_HandSoldering" H 3338 1800 50  0001 C CNN
+F 2 "Capacitors_SMD:C_0805_HandSoldering" H 3338 1800 50  0001 C CNN
 F 3 "" H 3300 1950 50  0000 C CNN
 	1    3300 1950
@@
 F 0 "C18" H 3525 2050 50  0000 L CNN
 F 1 "1uF" V 3450 1750 50  0000 L CNN
-F 2 "Capacitors_SMD:C_0603_HandSoldering" H 3538 1800 50  0001 C CNN
+F 2 "Capacitors_SMD:C_0805_HandSoldering" H 3538 1800 50  0001 C CNN
 F 3 "" H 3500 1950 50  0000 C CNN
 	1    3500 1950
@@
 F 0 "C13" H 2425 1850 50  0000 L CNN
 F 1 "100nF" V 2350 1450 50  0000 L CNN
-F 2 "Capacitors_SMD:C_0603_HandSoldering" H 2438 1600 50  0001 C CNN
+F 2 "Capacitors_SMD:C_0805_HandSoldering" H 2438 1600 50  0001 C CNN
 F 3 "" H 2400 1750 50  0000 C CNN
 	1    2400 1750
@@
 F 0 "C14" H 2625 1850 50  0000 L CNN
 F 1 "1uF" V 2550 1550 50  0000 L CNN
-F 2 "Capacitors_SMD:C_0603_HandSoldering" H 2638 1600 50  0001 C CNN
+F 2 "Capacitors_SMD:C_0805_HandSoldering" H 2638 1600 50  0001 C CNN
 F 3 "" H 2600 1750 50  0000 C CNN
 	1    2600 1750
@@
 F 0 "C16" H 3075 1950 50  0000 L CNN
 F 1 "1uF" V 3000 1650 50  0000 L CNN
-F 2 "Capacitors_SMD:C_0603_HandSoldering" H 3088 1700 50  0001 C CNN
+F 2 "Capacitors_SMD:C_0805_HandSoldering" H 3088 1700 50  0001 C CNN
 F 3 "" H 3050 1850 50  0000 C CNN
 	1    3050 1850
@@
 F 0 "C15" H 2875 1950 50  0000 L CNN
 F 1 "100nF" V 2800 1550 50  0000 L CNN
-F 2 "Capacitors_SMD:C_0603_HandSoldering" H 2888 1700 50  0001 C CNN
+F 2 "Capacitors_SMD:C_0805_HandSoldering" H 2888 1700 50  0001 C CNN
 F 3 "" H 2850 1850 50  0000 C CNN
 	1    2850 1850
@@
 F 0 "BT1" H 2050 2900 50  0000 L CNN
 F 1 "CR_BAT" H 2050 2800 50  0000 L CNN
-F 2 "" V 1950 2860 50  0001 C CNN
+F 2 "Battery_Holders:BatteryHolder_CoinCell_Keystone_3008" V 1950 2860 50  0001 C CNN
 F 3 "" V 1950 2860 50  0000 C CNN
 	1    1950 2800
@@
 F 0 "C8" H 2025 4300 50  0000 L CNN
 F 1 "100nF" V 1950 3900 50  0000 L CNN
-F 2 "Capacitors_SMD:C_0603_HandSoldering" H 2038 4050 50  0001 C CNN
+F 2 "Capacitors_SMD:C_0805_HandSoldering" H 2038 4050 50  0001 C CNN
 F 3 "" H 2000 4200 50  0000 C CNN
 	1    2000 4200
@@
 F 0 "C11" H 2325 4300 50  0000 L CNN
 F 1 "1uF" H 2350 4100 50  0000 L CNN
-F 2 "Capacitors_SMD:C_0603_HandSoldering" H 2338 4050 50  0001 C CNN
+F 2 "Capacitors_SMD:C_0805_HandSoldering" H 2338 4050 50  0001 C CNN
 F 3 "" H 2300 4200 50  0000 C CNN
 	1    2300 4200
@@
 F 0 "C9" H 2075 5850 50  0000 L CNN
 F 1 "100nF" V 2000 5450 50  0000 L CNN
-F 2 "Capacitors_SMD:C_0603_HandSoldering" H 2088 5600 50  0001 C CNN
+F 2 "Capacitors_SMD:C_0805_HandSoldering" H 2088 5600 50  0001 C CNN
 F 3 "" H 2050 5750 50  0000 C CNN
 	1    2050 5750
@@
 F 0 "C12" H 2375 5850 50  0000 L CNN
 F 1 "1uF" H 2400 5650 50  0000 L CNN
-F 2 "Capacitors_SMD:C_0603_HandSoldering" H 2388 5600 50  0001 C CNN
+F 2 "Capacitors_SMD:C_0805_HandSoldering" H 2388 5600 50  0001 C CNN
 F 3 "" H 2350 5750 50  0000 C CNN
 	1    2350 5750
