File: AriG25Module.sch (KiCad schematic (older format))
At the start: 17 parts, among them J1 CON, U2 ARIA-G25

Commit message: Schematic changes. PCB in process of making.
Removed LAN9500A Jtag. Removed Aria G25 pinout. Removed USB connectors. Added rezistors to USB/ETH/ySD shields.
Parts:
- removed J1: CON, symbol HEADER_15x2
- BT1: footprint Battery_Holders:BatteryHolder_CoinCell_Keystone_3008 -> Battery_Holders:BatteryHolder_CoinCell_Keystone_3001
- L2: footprint (none) -> Resistors_SMD:R_0603_HandSoldering
- S1: footprint (none) -> Buttons_Switches_SMD:SW_SPST_EVPBF
- U2: footprint (none) -> misc:ARIA-G25
Connections:
- net labels added: PC31
- wire segments 152 -> 122
Changed lines of the file:
@@
 $Descr A4 11693 8268
 encoding utf-8
-Sheet 7 7
+Sheet 3 7
 Title ""
 Date ""
@@
 F 0 "U2" H 4150 7050 60  0000 L BNB
 F 1 "ARIA-G25" H 4150 1250 40  0000 L TNN
-F 2 "" H 4150 1150 40  0001 L CNN
+F 2 "misc:ARIA-G25" H 4150 1150 40  0001 L CNN
 F 3 "" H 2200 5800 60  0001 C CNN
 F 4 "IC" H 4150 7150 40  0001 L BNN "Family"
@@
 $EndComp
 $Comp
-L GND #PWR015
+L GND #PWR013
 U 1 1 587D3F4F
 P 2050 1900
-F 0 "#PWR015" H 2050 1650 50  0001 C CNN
+F 0 "#PWR013" H 2050 1650 50  0001 C CNN
 F 1 "GND" H 2050 1750 50  0000 C CNN
 F 2 "" H 2050 1900 50  0000 C CNN
@@
 $EndComp
 $Comp
-L GND #PWR016
+L GND #PWR014
 U 1 1 587D3F7C
 P 2500 2000
-F 0 "#PWR016" H 2500 1750 50  0001 C CNN
+F 0 "#PWR014" H 2500 1750 50  0001 C CNN
 F 1 "GND" H 2500 1850 50  0000 C CNN
 F 2 "" H 2500 2000 50  0000 C CNN
@@
 $EndComp
 $Comp
-L GND #PWR017
+L GND #PWR015
 U 1 1 587D3FA2
 P 2950 2100
-F 0 "#PWR017" H 2950 1850 50  0001 C CNN
+F 0 "#PWR015" H 2950 1850 50  0001 C CNN
 F 1 "GND" H 2950 1950 50  0000 C CNN
 F 2 "" H 2950 2100 50  0000 C CNN
@@
 $EndComp
 $Comp
-L GND #PWR018
+L GND #PWR016
 U 1 1 587D3FC8
 P 3400 2200
-F 0 "#PWR018" H 3400 1950 50  0001 C CNN
+F 0 "#PWR016" H 3400 1950 50  0001 C CNN
 F 1 "GND" H 3400 2050 50  0000 C CNN
 F 2 "" H 3400 2200 50  0000 C CNN
@@
 $EndComp
 $Comp
-L +3.3V #PWR019
+L +3.3V #PWR017
 U 1 1 587D41CA
 P 3500 1300
-F 0 "#PWR019" H 3500 1150 50  0001 C CNN
+F 0 "#PWR017" H 3500 1150 50  0001 C CNN
 F 1 "+3.3V" H 3500 1440 50  0000 C CNN
 F 2 "" H 3500 1300 50  0000 C CNN
@@
 $EndComp
 $Comp
-L GND #PWR020
+L GND #PWR018
 U 1 1 587D4706
 P 3900 7000
-F 0 "#PWR020" H 3900 6750 50  0001 C CNN
+F 0 "#PWR018" H 3900 6750 50  0001 C CNN
 F 1 "GND" H 3900 6850 50  0000 C CNN
 F 2 "" H 3900 7000 50  0000 C CNN
@@
 F 0 "BT1" H 2050 2900 50  0000 L CNN
 F 1 "CR_BAT" H 2050 2800 50  0000 L CNN
-F 2 "Battery_Holders:BatteryHolder_CoinCell_Keystone_3008" V 1950 2860 50  0001 C CNN
+F 2 "Battery_Holders:BatteryHolder_CoinCell_Keystone_3001" V 1950 2860 50  0001 C CNN
 F 3 "" V 1950 2860 50  0000 C CNN
 	1    1950 2800
@@
 VBAT
 $Comp
-L GND #PWR021
+L GND #PWR019
 U 1 1 58979EE3
 P 1950 3000
-F 0 "#PWR021" H 1950 2750 50  0001 C CNN
+F 0 "#PWR019" H 1950 2750 50  0001 C CNN
 F 1 "GND" H 1950 2850 50  0000 C CNN
 F 2 "" H 1950 3000 50  0000 C CNN
@@
 F 0 "S1" V 1850 4100 60  0000 C CNN
 F 1 "~RST" V 1700 4100 60  0000 C CNN
-F 2 "" H 1750 4250 60  0001 C CNN
+F 2 "Buttons_Switches_SMD:SW_SPST_EVPBF" H 1750 4250 60  0001 C CNN
 F 3 "" H 1750 4250 60  0000 C CNN
 	1    1750 4250
@@
 $EndComp
 $Comp
-L +3.3V #PWR022
+L +3.3V #PWR020
 U 1 1 5897B046
 P 1750 3900
-F 0 "#PWR022" H 1750 3750 50  0001 C CNN
+F 0 "#PWR020" H 1750 3750 50  0001 C CNN
 F 1 "+3.3V" H 1750 4040 50  0000 C CNN
 F 2 "" H 1750 3900 50  0000 C CNN
@@
 $EndComp
 $Comp
-L GND #PWR023
+L GND #PWR021
 U 1 1 5897B24B
 P 2150 4500
-F 0 "#PWR023" H 2150 4250 50  0001 C CNN
+F 0 "#PWR021" H 2150 4250 50  0001 C CNN
 F 1 "GND" H 2150 4350 50  0000 C CNN
 F 2 "" H 2150 4500 50  0000 C CNN
@@
 $EndComp
 $Comp
-L GND #PWR024
+L GND #PWR022
 U 1 1 5897B2E1
 P 1750 4600
-F 0 "#PWR024" H 1750 4350 50  0001 C CNN
+F 0 "#PWR022" H 1750 4350 50  0001 C CNN
 F 1 "GND" H 1750 4450 50  0000 C CNN
 F 2 "" H 1750 4600 50  0000 C CNN
@@
 $EndComp
 $Comp
-L GND #PWR025
+L GND #PWR023
 U 1 1 589CDFC4
 P 2200 6050
-F 0 "#PWR025" H 2200 5800 50  0001 C CNN
+F 0 "#PWR023" H 2200 5800 50  0001 C CNN
 F 1 "GND" H 2200 5900 50  0000 C CNN
 F 2 "" H 2200 6050 50  0000 C CNN
@@
 Connection ~ 2200 5950
 $Comp
-L +3.3V #PWR026
+L +3.3V #PWR024
 U 1 1 589CE2E5
 P 2050 5400
-F 0 "#PWR026" H 2050 5250 50  0001 C CNN
+F 0 "#PWR024" H 2050 5250 50  0001 C CNN
 F 1 "+3.3V" H 2050 5540 50  0000 C CNN
 F 2 "" H 2050 5400 50  0000 C CNN
@@
 Wire Wire Line
 	5650 6900 5750 6900
-Text Label 8250 1500 2    50   ~ 0
-AD0
-Text Label 8750 1500 0    50   ~ 0
-AD1
-Text Label 8250 1600 2    50   ~ 0
-AD2
-Text Label 8750 1600 0    50   ~ 0
-AD3
-Wire Wire Line
-	8250 1500 8350 1500
-Wire Wire Line
-	8650 1500 8750 1500
-Wire Wire Line
-	8250 1600 8350 1600
-Wire Wire Line
-	8650 1600 8750 1600
 Text Label 3900 5600 2    50   ~ 0
 SDA0
@@
 Wire Wire Line
 	3900 5700 4000 5700
-Text Label 8250 1700 2    50   ~ 0
-SDA0
-Wire Wire Line
-	8250 1700 8350 1700
-Text Label 8250 1800 2    50   ~ 0
-SCL0
-Wire Wire Line
-	8250 1800 8350 1800
-Text HLabel 8750 1700 2    50   Input ~ 0
-TXD0
-Text HLabel 8750 1800 2    50   Input ~ 0
-RXD0
-Wire Wire Line
-	8650 1700 8750 1700
-Wire Wire Line
-	8650 1800 8750 1800
 Text Label 5750 2200 0    50   ~ 0
 SDA1
@@
 Wire Wire Line
 	5650 2300 5750 2300
-Text Label 8250 2000 2    50   ~ 0
-SCL1
-Text HLabel 8750 1900 2    50   Input ~ 0
-TXD1
-Text HLabel 8750 2000 2    50   Input ~ 0
-RXD1
 Text Label 3900 3500 2    50   ~ 0
 MISO
@@
 Wire Wire Line
 	3900 3800 4000 3800
-Text Label 8250 2100 2    50   ~ 0
-MISO
-Text Label 8250 2200 2    50   ~ 0
-MOSI
-Text Label 8750 2100 0    50   ~ 0
-SPCK
-Text Label 8750 2200 0    50   ~ 0
-NPCS0
 Text Label 5750 4200 0    50   ~ 0
 PWM0
@@
 Wire Wire Line
 	5650 4500 5750 4500
-Text Label 8250 2300 2    50   ~ 0
-PWM0
-Text Label 8750 2300 0    50   ~ 0
-PWM1
-Text Label 8250 2400 2    50   ~ 0
-PWM2
-Text Label 8750 2400 0    50   ~ 0
-PWM3
 Text Label 3900 4600 2    50   ~ 0
 1W
 Wire Wire Line
 	3900 4600 4000 4600
-Text Label 8250 2500 2    50   ~ 0
-1W
 Text Label 5750 3100 0    50   ~ 0
 PC8
@@
 Wire Wire Line
 	5650 3400 5750 3400
-Text Label 8250 2600 2    50   ~ 0
-PC8
-Text Label 8750 2600 0    50   ~ 0
-PC9
-Text Label 8250 2700 2    50   ~ 0
-PC10
-Text Label 8750 2700 0    50   ~ 0
-PC11
-Text Label 8250 1900 2    50   ~ 0
-SDA1
-$Comp
-L GND #PWR027
-U 1 1 589E02C3
-P 8250 3000
-F 0 "#PWR027" H 8250 2750 50  0001 C CNN
-F 1 "GND" H 8250 2850 50  0000 C CNN
-F 2 "" H 8250 3000 50  0000 C CNN
-F 3 "" H 8250 3000 50  0000 C CNN
-	1    8250 3000
-	1    0    0    -1
-$EndComp
-Wire Wire Line
-	8250 2800 8250 3000
-Wire Wire Line
-	8250 2900 8350 2900
-Wire Wire Line
-	8250 2800 8350 2800
-Connection ~ 8250 2900
-Wire Wire Line
-	8250 2700 8350 2700
-Wire Wire Line
-	8250 2600 8350 2600
-Wire Wire Line
-	8250 2500 8350 2500
-Wire Wire Line
-	8250 2400 8350 2400
-Wire Wire Line
-	8250 2300 8350 2300
-Wire Wire Line
-	8250 2200 8350 2200
-Wire Wire Line
-	8250 2100 8350 2100
-Wire Wire Line
-	8250 2000 8350 2000
-Wire Wire Line
-	8250 1900 8350 1900
-Wire Wire Line
-	8650 2700 8750 2700
-Wire Wire Line
-	8650 2600 8750 2600
-Wire Wire Line
-	8650 2400 8750 2400
-Wire Wire Line
-	8650 2300 8750 2300
-Wire Wire Line
-	8650 2200 8750 2200
-Wire Wire Line
-	8650 2100 8750 2100
-Wire Wire Line
-	8650 2000 8750 2000
-Wire Wire Line
-	8650 1900 8750 1900
-$Comp
-L GND #PWR028
-U 1 1 589E162A
-P 8750 3000
-F 0 "#PWR028" H 8750 2750 50  0001 C CNN
-F 1 "GND" H 8750 2850 50  0000 C CNN
-F 2 "" H 8750 3000 50  0000 C CNN
-F 3 "" H 8750 3000 50  0000 C CNN
-	1    8750 3000
-	1    0    0    -1
-$EndComp
-$Comp
-L HEADER_15x2 J1
-U 1 1 589E1657
-P 8500 2200
-F 0 "J1" H 8500 3000 60  0000 C CNN
-F 1 "CON" H 8500 1400 60  0000 C CNN
-F 2 "" H 8500 2200 60  0001 C CNN
-F 3 "" H 8500 2200 60  0000 C CNN
-	1    8500 2200
-	1    0    0    -1
-$EndComp
-Wire Wire Line
-	8650 2900 8750 2900
-Wire Wire Line
-	8750 2800 8750 3000
-Wire Wire Line
-	8650 2800 8750 2800
-Connection ~ 8750 2900
 $Comp
 L L_Core_Iron_Small L2
@@
 F 0 "L2" H 2600 5540 50  0000 L CNN
 F 1 "LF" H 2600 5450 50  0000 L CNN
-F 2 "" H 2550 5500 50  0001 C CNN
+F 2 "Resistors_SMD:R_0603_HandSoldering" H 2550 5500 50  0001 C CNN
 F 3 "" H 2550 5500 50  0000 C CNN
 	1    2550 5500
@@
 	2700 5500 2650 5500
 $Comp
-L +3.3V #PWR029
+L +3.3V #PWR025
 U 1 1 58A03E70
 P 6300 6100
-F 0 "#PWR029" H 6300 5950 50  0001 C CNN
+F 0 "#PWR025" H 6300 5950 50  0001 C CNN
 F 1 "+3.3V" H 6300 6240 50  0000 C CNN
 F 2 "" H 6300 6100 50  0000 C CNN
@@
 <-- ???
 $Comp
-L PWR_FLAG #FLG030
+L PWR_FLAG #FLG026
 U 1 1 58A0D352
 P 1850 2500
-F 0 "#FLG030" H 1850 2595 50  0001 C CNN
+F 0 "#FLG026" H 1850 2595 50  0001 C CNN
 F 1 "PWR_FLAG" H 1850 2680 50  0000 C CNN
 F 2 "" H 1850 2500 50  0000 C CNN
@@
 Wire Wire Line
 	3900 6100 4000 6100
+Text HLabel 5750 5600 2    50   BiDi ~ 0
+PC31
+Wire Wire Line
+	5650 5600 5750 5600
 $EndSCHEMATC

Commit message: Modified USB/ETH label names.
Connections:
- net ETHRXN renamed ETHRX_N
- net ETHRXP renamed ETHRX_P
- net ETHTXN renamed ETHTX_N
- net ETHTXP renamed ETHTX_P
- net USBAN renamed USBA_N
- net USBAP renamed USBA_P
- net USBBN renamed USBB_N
- net USBBP renamed USBB_P
- net USBCN renamed USBC_N
- net USBCP renamed USBC_P
Changed lines of the file:
@@
 DTXD
 Text HLabel 5750 5800 2    50   Input ~ 0
-ETHRXP
+ETHRX_P
 Text HLabel 5750 5900 2    50   Input ~ 0
-ETHRXN
+ETHRX_N
 Text HLabel 5750 6000 2    50   Output ~ 0
-ETHTXP
+ETHTX_P
 Text HLabel 5750 6100 2    50   Output ~ 0
-ETHTXN
+ETHTX_N
 Text HLabel 6400 6200 2    50   Output ~ 0
 ETH3V3
@@
 RXD3
 Text HLabel 5750 1800 2    50   BiDi ~ 0
-USBAP
+USBA_P
 Text HLabel 5750 1900 2    50   BiDi ~ 0
-USBAN
+USBA_N
 Text HLabel 5750 4900 2    50   BiDi ~ 0
 PC24
@@
 VBAT
 Text HLabel 5750 1700 2    50   BiDi ~ 0
-USBBN
+USBB_N
 Text HLabel 5750 1600 2    50   BiDi ~ 0
-USBBP
+USBB_P
 Text HLabel 5750 1400 2    50   BiDi ~ 0
-USBCP
+USBC_P
 Text HLabel 5750 1500 2    50   BiDi ~ 0
-USBCN
+USBC_N
 $Comp
 L SW_TACT S1

Commit message: Finished first version of PCB.
Modified RJ45 footprint.
Parts:
- added R17: 1k, Resistors_SMD:R_0603_HandSoldering, symbol R
- S1: footprint Buttons_Switches_SMD:SW_SPST_EVPBF -> misc:SW_SPST_EVPBF
Connections:
- net +3V3: now also R17.1; no longer C11.1, C8.1, S1.1, S1.2, U2.E21 (~NRST)
- new net ~RST: C11.1, C8.1, R17.2, S1.1, S1.2, U2.E21 (~NRST)
Changed lines of the file:
@@
 F 0 "S1" V 1850 4100 60  0000 C CNN
 F 1 "~RST" V 1700 4100 60  0000 C CNN
-F 2 "Buttons_Switches_SMD:SW_SPST_EVPBF" H 1750 4250 60  0001 C CNN
+F 2 "misc:SW_SPST_EVPBF" H 1750 4250 60  0001 C CNN
 F 3 "" H 1750 4250 60  0000 C CNN
 	1    1750 4250
@@
 L +3.3V #PWR020
 U 1 1 5897B046
-P 1750 3900
-F 0 "#PWR020" H 1750 3750 50  0001 C CNN
-F 1 "+3.3V" H 1750 4040 50  0000 C CNN
-F 2 "" H 1750 3900 50  0000 C CNN
-F 3 "" H 1750 3900 50  0000 C CNN
-	1    1750 3900
+P 1750 3450
+F 0 "#PWR020" H 1750 3300 50  0001 C CNN
+F 1 "+3.3V" H 1750 3590 50  0000 C CNN
+F 2 "" H 1750 3450 50  0000 C CNN
+F 3 "" H 1750 3450 50  0000 C CNN
+	1    1750 3450
 	1    0    0    -1
 $EndComp
@@
 	1700 3950 2400 3950
 Wire Wire Line
-	1750 3950 1750 3900
+	1750 3850 1750 3950
 Wire Wire Line
 	1800 3950 1800 4000
@@
 Wire Wire Line
 	5650 5600 5750 5600
+$Comp
+L R R17
+U 1 1 58B5772C
+P 1750 3700
+F 0 "R17" V 1830 3700 50  0000 C CNN
+F 1 "1k" V 1750 3700 50  0000 C CNN
+F 2 "Resistors_SMD:R_0603_HandSoldering" V 1680 3700 50  0001 C CNN
+F 3 "" H 1750 3700 50  0000 C CNN
+	1    1750 3700
+	1    0    0    -1
+$EndComp
+Wire Wire Line
+	1750 3550 1750 3450
 $EndSCHEMATC

Commit message: Modified buck circuit on board.
Parts:
- C10, C11, C12, C13, C14, C15, C16, C17, C18, C7, C8, C9: footprint Capacitors_SMD:C_0805_HandSoldering -> Capacitors_SMD:C_0603_HandSoldering
Changed lines of the file:
@@
 F 0 "C10" H 2175 1750 50  0000 L CNN
 F 1 "1uF" V 2100 1450 50  0000 L CNN
-F 2 "Capacitors_SMD:C_0805_HandSoldering" H 2188 1500 50  0001 C CNN
+F 2 "Capacitors_SMD:C_0603_HandSoldering" H 2188 1500 50  0001 C CNN
 F 3 "" H 2150 1650 50  0000 C CNN
 	1    2150 1650
@@
 F 0 "C7" H 1975 1750 50  0000 L CNN
 F 1 "100nF" V 1900 1400 50  0000 L CNN
-F 2 "Capacitors_SMD:C_0805_HandSoldering" H 1988 1500 50  0001 C CNN
+F 2 "Capacitors_SMD:C_0603_HandSoldering" H 1988 1500 50  0001 C CNN
 F 3 "" H 1950 1650 50  0000 C CNN
 	1    1950 1650
@@
 F 0 "C17" H 3325 2050 50  0000 L CNN
 F 1 "100nF" V 3250 1650 50  0000 L CNN
-F 2 "Capacitors_SMD:C_0805_HandSoldering" H 3338 1800 50  0001 C CNN
+F 2 "Capacitors_SMD:C_0603_HandSoldering" H 3338 1800 50  0001 C CNN
 F 3 "" H 3300 1950 50  0000 C CNN
 	1    3300 1950
@@
 F 0 "C18" H 3525 2050 50  0000 L CNN
 F 1 "1uF" V 3450 1750 50  0000 L CNN
-F 2 "Capacitors_SMD:C_0805_HandSoldering" H 3538 1800 50  0001 C CNN
+F 2 "Capacitors_SMD:C_0603_HandSoldering" H 3538 1800 50  0001 C CNN
 F 3 "" H 3500 1950 50  0000 C CNN
 	1    3500 1950
@@
 F 0 "C13" H 2425 1850 50  0000 L CNN
 F 1 "100nF" V 2350 1450 50  0000 L CNN
-F 2 "Capacitors_SMD:C_0805_HandSoldering" H 2438 1600 50  0001 C CNN
+F 2 "Capacitors_SMD:C_0603_HandSoldering" H 2438 1600 50  0001 C CNN
 F 3 "" H 2400 1750 50  0000 C CNN
 	1    2400 1750
@@
 F 0 "C14" H 2625 1850 50  0000 L CNN
 F 1 "1uF" V 2550 1550 50  0000 L CNN
-F 2 "Capacitors_SMD:C_0805_HandSoldering" H 2638 1600 50  0001 C CNN
+F 2 "Capacitors_SMD:C_0603_HandSoldering" H 2638 1600 50  0001 C CNN
 F 3 "" H 2600 1750 50  0000 C CNN
 	1    2600 1750
@@
 F 0 "C16" H 3075 1950 50  0000 L CNN
 F 1 "1uF" V 3000 1650 50  0000 L CNN
-F 2 "Capacitors_SMD:C_0805_HandSoldering" H 3088 1700 50  0001 C CNN
+F 2 "Capacitors_SMD:C_0603_HandSoldering" H 3088 1700 50  0001 C CNN
 F 3 "" H 3050 1850 50  0000 C CNN
 	1    3050 1850
@@
 F 0 "C15" H 2875 1950 50  0000 L CNN
 F 1 "100nF" V 2800 1550 50  0000 L CNN
-F 2 "Capacitors_SMD:C_0805_HandSoldering" H 2888 1700 50  0001 C CNN
+F 2 "Capacitors_SMD:C_0603_HandSoldering" H 2888 1700 50  0001 C CNN
 F 3 "" H 2850 1850 50  0000 C CNN
 	1    2850 1850
@@
 F 0 "C8" H 2025 4300 50  0000 L CNN
 F 1 "100nF" V 1950 3900 50  0000 L CNN
-F 2 "Capacitors_SMD:C_0805_HandSoldering" H 2038 4050 50  0001 C CNN
+F 2 "Capacitors_SMD:C_0603_HandSoldering" H 2038 4050 50  0001 C CNN
 F 3 "" H 2000 4200 50  0000 C CNN
 	1    2000 4200
@@
 F 0 "C11" H 2325 4300 50  0000 L CNN
 F 1 "1uF" H 2350 4100 50  0000 L CNN
-F 2 "Capacitors_SMD:C_0805_HandSoldering" H 2338 4050 50  0001 C CNN
+F 2 "Capacitors_SMD:C_0603_HandSoldering" H 2338 4050 50  0001 C CNN
 F 3 "" H 2300 4200 50  0000 C CNN
 	1    2300 4200
@@
 F 0 "C9" H 2075 5850 50  0000 L CNN
 F 1 "100nF" V 2000 5450 50  0000 L CNN
-F 2 "Capacitors_SMD:C_0805_HandSoldering" H 2088 5600 50  0001 C CNN
+F 2 "Capacitors_SMD:C_0603_HandSoldering" H 2088 5600 50  0001 C CNN
 F 3 "" H 2050 5750 50  0000 C CNN
 	1    2050 5750
@@
 F 0 "C12" H 2375 5850 50  0000 L CNN
 F 1 "1uF" H 2400 5650 50  0000 L CNN
-F 2 "Capacitors_SMD:C_0805_HandSoldering" H 2388 5600 50  0001 C CNN
+F 2 "Capacitors_SMD:C_0603_HandSoldering" H 2388 5600 50  0001 C CNN
 F 3 "" H 2350 5750 50  0000 C CNN
 	1    2350 5750

Commit message: Modified schematic. v1.1
Parts:
- removed C11: 1uF, Capacitors_SMD:C_0603_HandSoldering, symbol C
- removed C9: 100nF, Capacitors_SMD:C_0603_HandSoldering, symbol C
- removed L2: LF, Resistors_SMD:R_0603_HandSoldering, symbol L_Core_Iron_Small
- removed S1: ~RST, misc:SW_SPST_EVPBF, symbol SW_TACT
- added C22, C24: 100nF, Capacitors_SMD:C_0603_HandSoldering, symbol C
- added D5: LED, LEDs:LED_0603, symbol LED
- added D6: TL431DBZ, TO_SOT_Packages_SMD:SOT-23, symbol TL431DBZ
- added R11, R12, R13, R14, R15, R16, R17, R18, R9: R, Resistors_SMD:R_0603_HandSoldering, symbol R
- added SW1: BTN, Buttons_Switches_SMD:SW_SPST_EVQPE1, symbol SW_DPST_x2
- added SW2: ~RST, Buttons_Switches_SMD:SW_SPST_EVQPE1, symbol SW_DPST_x2
- added W10: RXD2_T, Measurement_Points:Measurement_Point_Round-SMD-Pad_Small, symbol TEST_1P
- added W11: TXD3_T, Measurement_Points:Measurement_Point_Round-SMD-Pad_Small, symbol TEST_1P
- added W12: RXD3_T, Measurement_Points:Measurement_Point_Round-SMD-Pad_Small, symbol TEST_1P
- added W13: DRXD_T, Measurement_Points:Measurement_Point_Round-SMD-Pad_Small, symbol TEST_1P
- added W14: DTXD_T, Measurement_Points:Measurement_Point_Round-SMD-Pad_Small, symbol TEST_1P
- added W5: TXD0_T, Measurement_Points:Measurement_Point_Round-SMD-Pad_Small, symbol TEST_1P
- added W6: RXD0_T, Measurement_Points:Measurement_Point_Round-SMD-Pad_Small, symbol TEST_1P
- added W7: TXD1_T, Measurement_Points:Measurement_Point_Round-SMD-Pad_Small, symbol TEST_1P
- added W8: RXD1_T, Measurement_Points:Measurement_Point_Round-SMD-Pad_Small, symbol TEST_1P
- added W9: TXD2_T, Measurement_Points:Measurement_Point_Round-SMD-Pad_Small, symbol TEST_1P
- C26: renamed from C12; value 1uF -> 10uF
- R10: renamed from R17; value 1k -> 10k
- renumbered C7 to C15, C10 to C16, C13 to C17, C14 to C18, C15 to C19, C16 to C20, C17 to C21, C18 to C23, C8 to C25, U2 to U3
Connections:
- net ADVREF is gone; now on net +3V3: U3.W19 (ADVREF)
- net +3V3: now also D6.1 (K), D6.2 (REF), R11.1; no longer U3.W6 (ETH3V3)
- net DRXD: now also W13.1
- net DTXD: now also W14.1
- net GND: now also C22.1, C24.1, D5.1 (K), D6.3 (A), R12.2, R14.2, R16.2, R18.2, SW1.2 (B), SW2.2 (B)
- net RXD0: now also W6.1
- net RXD1: now also W8.1
- net RXD2: now also W10.1
- net RXD3: now also W12.1
- net TXD0: now also W5.1
- net TXD1: now also W7.1
- net TXD2: now also W9.1
- net TXD3: now also W11.1
- net ~RST: now also SW2.1 (A)
- net PC30: now reaches U3.E10 (PC30)
- net at U3.E22 (~SHDN): now also C22.2
- net at U3.E23 (~WKUP): now also C24.2
- net CTS1: now reaches U3.E8 (CTS1/PC28)
- net PC29: now reaches U3.E9 (PC29)
- net 1W renamed 1WIRE
- net AD0 renamed 3V3_DIV
- net 3V3_DIV: now also R11.2, R12.1
- net AD1 renamed 5V_DIV
- net 5V_DIV: now also R13.2, R14.1
- net AD2 renamed VBUS_DIV
- net VBUS_DIV: now also R15.2, R16.1
- net AD3 renamed VIN_DIV
- net VIN_DIV: now also R17.2, R18.1
- net MISO: no longer names the net of U3.S12 (MISO/PA11)
- net MISO: now also R9.1
- net MOSI: no longer names the net of U3.S11 (MOSI/PA12)
- net MOSI: now also SW1.1 (A)
- net NPCS0: no longer names the net of U3.S9 (NPCS0/PA14)
- net PA2 renamed RTS0
- net PA3 renamed CTS0
- net PA4: no longer names the net of U3.S19 (PA4)
- net PC10: no longer names the net of U3.N12 (PC10)
- net PC11: no longer names the net of U3.N13 (PC11)
- net PC24 renamed RTS3
- net PC25 renamed CTS3
- net PC27 renamed RTS1
- net PC8: no longer names the net of U3.N10 (PC8/UTXD0)
- net PC9: no longer names the net of U3.N11 (PC9/URXD0)
- net PWM0: no longer names the net of U3.N20 (PC18/PWM0)
- net PWM1: no longer names the net of U3.N21 (PC19/PWM1)
- net PWM2: no longer names the net of U3.N22 (PC20/PWM2)
- net PWM3: no longer names the net of U3.N23 (PC21/PWM3)
- net SCL0: no longer names the net of U3.W18 (SCL0/PA31)
- net SCL1: no longer names the net of U3.N3 (PC1/SCL1)
- net SDA0: no longer names the net of U3.W17 (SDA0/PA30)
- net SDA1: no longer names the net of U3.N2 (PC0/SDA1)
- net SPCK: no longer names the net of U3.S10 (SPCK/PA13)
- new net: D5.2 (A), R9.2
- new net +5V: R13.1
- new net ETH3V3: U3.W6 (ETH3V3)
- new net VBUS: R15.1
- new net VIN: R17.1
- no-connect marks 0 -> 35
Other:
- note added: "Pull up ? ->"
- note added: "R??"
- note removed: "<-- ???"
- moved on the sheet: BT1, C15, C16, C17, C18, C19, C20, C21, C23, C25, C26, R10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
