File: Power.sch (KiCad schematic (older format))
At the start: 17 parts, among them CON1 PWR_JACK, P1 PWR_USB, U1 MCP16312-E/MS

Commit message: Modified LAN9500A schematic.
Modified the schematic for the USB to Ethernet converter.
Parts:
- C1, C2, C3, C4, C5, C6: footprint Capacitors_SMD:C_0603_HandSoldering -> Capacitors_SMD:C_0805_HandSoldering
- D3: footprint (none) -> LEDs:LED_0805
- R1, R2, R3: footprint Resistors_SMD:R_0603_HandSoldering -> Resistors_SMD:R_0805_HandSoldering
Changed lines of the file:
@@
 F 0 "C3" H 5650 3050 50  0000 L CNN
 F 1 "1uF" H 5800 3050 50  0000 L CNN
-F 2 "Capacitors_SMD:C_0603_HandSoldering" H 5788 2800 50  0001 C CNN
+F 2 "Capacitors_SMD:C_0805_HandSoldering" H 5788 2800 50  0001 C CNN
 F 3 "" H 5750 2950 50  0000 C CNN
 	1    5750 2950
@@
 F 0 "C1" H 5200 2850 50  0000 L CNN
 F 1 "10uF" H 5100 2650 50  0000 L CNN
-F 2 "Capacitors_SMD:C_0603_HandSoldering" H 5338 2600 50  0001 C CNN
+F 2 "Capacitors_SMD:C_0805_HandSoldering" H 5338 2600 50  0001 C CNN
 F 3 "" H 5300 2750 50  0000 C CNN
 	1    5300 2750
@@
 F 0 "C2" H 5450 2850 50  0000 L CNN
 F 1 "10uF" H 5350 2650 50  0000 L CNN
-F 2 "Capacitors_SMD:C_0603_HandSoldering" H 5588 2600 50  0001 C CNN
+F 2 "Capacitors_SMD:C_0805_HandSoldering" H 5588 2600 50  0001 C CNN
 F 3 "" H 5550 2750 50  0000 C CNN
 	1    5550 2750
@@
 F 0 "R1" V 7980 2850 50  0000 C CNN
 F 1 "31k6" V 7800 2850 50  0000 C CNN
-F 2 "Resistors_SMD:R_0603_HandSoldering" V 7830 2850 50  0001 C CNN
+F 2 "Resistors_SMD:R_0805_HandSoldering" V 7830 2850 50  0001 C CNN
 F 3 "" H 7900 2850 50  0000 C CNN
 	1    7900 2850
@@
 F 0 "R2" V 7980 3250 50  0000 C CNN
 F 1 "10k" V 7800 3250 50  0000 C CNN
-F 2 "Resistors_SMD:R_0603_HandSoldering" V 7830 3250 50  0001 C CNN
+F 2 "Resistors_SMD:R_0805_HandSoldering" V 7830 3250 50  0001 C CNN
 F 3 "" H 7900 3250 50  0000 C CNN
 	1    7900 3250
@@
 F 0 "C4" V 7100 2550 50  0000 L CNN
 F 1 "100nF" V 7100 2250 50  0000 L CNN
-F 2 "Capacitors_SMD:C_0603_HandSoldering" H 7288 2350 50  0001 C CNN
+F 2 "Capacitors_SMD:C_0805_HandSoldering" H 7288 2350 50  0001 C CNN
 F 3 "" H 7250 2500 50  0000 C CNN
 	1    7250 2500
@@
 F 0 "C5" H 8175 2950 50  0000 L CNN
 F 1 "10uF" H 8175 2750 50  0000 L CNN
-F 2 "Capacitors_SMD:C_0603_HandSoldering" H 8188 2700 50  0001 C CNN
+F 2 "Capacitors_SMD:C_0805_HandSoldering" H 8188 2700 50  0001 C CNN
 F 3 "" H 8150 2850 50  0000 C CNN
 	1    8150 2850
@@
 F 0 "C6" H 8425 2950 50  0000 L CNN
 F 1 "10uF" H 8425 2750 50  0000 L CNN
-F 2 "Capacitors_SMD:C_0603_HandSoldering" H 8438 2700 50  0001 C CNN
+F 2 "Capacitors_SMD:C_0805_HandSoldering" H 8438 2700 50  0001 C CNN
 F 3 "" H 8400 2850 50  0000 C CNN
 	1    8400 2850
@@
 F 0 "D3" H 8750 2950 50  0000 C CNN
 F 1 "PWR_LED" H 8750 2750 50  0000 C CNN
-F 2 "" H 8750 2850 50  0001 C CNN
+F 2 "LEDs:LED_0805" H 8750 2850 50  0001 C CNN
 F 3 "" H 8750 2850 50  0000 C CNN
 	1    8750 2850
@@
 F 0 "R3" V 8830 3250 50  0000 C CNN
 F 1 "R" V 8750 3250 50  0000 C CNN
-F 2 "Resistors_SMD:R_0603_HandSoldering" V 8680 3250 50  0001 C CNN
+F 2 "Resistors_SMD:R_0805_HandSoldering" V 8680 3250 50  0001 C CNN
 F 3 "" H 8750 3250 50  0000 C CNN
 	1    8750 3250
