File: Interfaces.sch (KiCad schematic (older format))
At the start: 21 parts, among them CON2 Micro_SD_Card, CON3 RJ45-TRF-LED, P4 DEBUG, U3 MCP2200, Y1 16MHz

Commit message: Modified schematic. v1.1
Parts:
- removed W3: RX_T, Pin_Headers:Pin_Header_Straight_1x01_Pitch2.54mm, symbol TEST_1P
- removed W4: TX_T, Pin_Headers:Pin_Header_Straight_1x01_Pitch2.54mm, symbol TEST_1P
- added C29, C30, C31, C36: 1nF, Capacitors_SMD:C_0603_HandSoldering, symbol C
- added C72: 100nF, Capacitors_SMD:C_0603_HandSoldering, symbol C
- added J1: 1W_H, Pin_Headers:Pin_Header_Straight_1x02_Pitch1.27mm, symbol HEADER_2
- added P1: USB_A, Connect:USB_A, symbol USB_A
- added R21, R42: 10k, Resistors_SMD:R_0603_HandSoldering, symbol R
- added R22: 1M, Resistors_SMD:R_0603_HandSoldering, symbol R
- U4: renamed from U3; footprint Housings_SSOP:SSOP-20_5.3x7.2mm_Pitch0.65mm -> Housings_SSOP:SSOP-20_4.4x6.5mm_Pitch0.65mm
- renumbered C19 to C27, C20 to C28, C21 to C32, C22 to C33, C23 to C34, C24 to C35, CON3 to CON2, CON2 to CON3, D4 to D7, D5 to D8, P4 to P2, R15 to R19, R16 to R20, R4 to R23, R5 to R24, R19 to R25, W2 to W15
Connections:
- net +3V3: now also D7.2 (A), D8.2 (A), R21.1
- net GND: now also C29.1, C30.1, C31.1, C36.1, C72.2, J1.2, P1.4 (GND), R22.2; no longer D7.1 (K), D8.1 (K)
- net TCT: now also CON2.3 (TCT); no longer CON2.2 (TD-)
- net TD-: now also CON2.2 (TD-); no longer CON2.3 (TCT)
- net at CON3.9 (SHIELD), R20.2: now also C30.2
- net at U4.4 (~RST): now also C72.1, R42.1; no longer W15.1
- net at P2.6 (shield), R25.1: now also C36.2
- net at R23.2: now also D7.1 (K); no longer D7.2 (A)
- net at R24.2: now also D8.1 (K); no longer D8.2 (A)
- net at CON2.4 (SHIELD), CON2.5 (SHIELD), R19.1: now also C29.2
- new net: R42.2, W15.1
- new net: C31.2, P1.5 (shield), R22.1
- new net +5V: P1.1 (VBUS)
- new net 1WIRE: J1.1, R21.2
- new net USBD+: P1.3 (D+)
- new net USBD-: P1.2 (D-)
- no-connect marks 0 -> 9
Other:
- note added: "RC 10k 100n ->"
- note removed: "<- +condensator?"
- moved on the sheet: D7, D8, R19, W15
