File: Interfaces.sch (KiCad schematic (older format))
At the start: 29 parts, among them CON2 RJ45-TRF-LED, CON3 Micro_SD_Card, J1 1W_H, P1 USB_A, P2 DEBUG, U4 MCP2200, Y1 16MHz

Commit message: Modified board. v1.1 to reflect the schematic change.
Changed lines of the file:
@@
 Text HLabel 1650 5350 2    50   BiDi ~ 0
 nETH_USB_USBD+
-$Sheet
-S 950  5800 600  1000
-U 588F1A51
-F0 "SERIAL_RS232_conv" 50
-F1 "SERIAL_RS232_conv.sch" 50
-F2 "IN_TX" O R 1550 5900 50
-F3 "IN_RX" I R 1550 6000 50
-F4 "IN_CTS" I R 1550 6100 50
-F5 "IN_RTS" O R 1550 6200 50
-F6 "OUT_TX" O R 1550 6400 50
-F7 "OUT_RTS" O R 1550 6700 50
-F8 "OUT_RX" I R 1550 6500 50
-F9 "OUT_CTS" I R 1550 6600 50
-$EndSheet
 Text HLabel 1650 5900 2    50   Output ~ 0
 RS232_IN_TX
@@
 VBUS
 Wire Wire Line
-	9250 5050 9350 5050
-Wire Wire Line
 	9750 6150 9750 6050
 Wire Wire Line
@@
 RS232_IN_CTS
 Wire Wire Line
-	1650 6000 1550 6000
-Wire Wire Line
-	1550 5900 1650 5900
-Wire Wire Line
 	1550 6400 1650 6400
 Wire Wire Line
@@
 Text HLabel 1650 6200 2    50   Output ~ 0
 RS232_IN_RTS
-Wire Wire Line
-	1550 6100 1650 6100
-Wire Wire Line
-	1550 6200 1650 6200
 Text HLabel 1650 6600 2    50   Input ~ 0
 RS232_OUT_CTS
@@
 Wire Wire Line
 	4150 6500 4250 6500
+$Sheet
+S 950  5800 600  1000
+U 588F1A51
+F0 "SERIAL_RS232_conv" 50
+F1 "SERIAL_RS232_conv.sch" 50
+F2 "IN_TX" O R 1550 5900 50
+F3 "IN_RX" I R 1550 6000 50
+F4 "IN_RTS" O R 1550 6200 50
+F5 "OUT_TX" O R 1550 6400 50
+F6 "OUT_RTS" O R 1550 6700 50
+F7 "OUT_RX" I R 1550 6500 50
+F8 "OUT_CTS" I R 1550 6600 50
+F9 "IN_CTS" I R 1550 6100 50
+$EndSheet
+Wire Wire Line
+	1550 5900 1650 5900
+Wire Wire Line
+	1550 6000 1650 6000
+Wire Wire Line
+	1550 6100 1650 6100
+Wire Wire Line
+	1550 6200 1650 6200
+Wire Wire Line
+	9350 5050 9250 5050
 $EndSCHEMATC
