File: SERIAL_RS232_conv.sch (KiCad schematic (older format))
At the start: 9 parts, among them IC1 MAX3232, J4 MDB9_IN, J5 MDB9_OUT

Commit message: Modified schematic. v1.1
Parts:
- added C60: 100nF, Capacitors_SMD:C_0603_HandSoldering, symbol C
- added C61, C62, C63, C66, C67: 0.1uF, Capacitors_SMD:C_0603_HandSoldering, symbol C
- added IC2: MAX3232, Housings_SSOP:SSOP-16_3.9x4.9mm_Pitch0.635mm, symbol MAX3232
- IC1: footprint SMD_Packages:SO-16-L -> Housings_SSOP:SSOP-16_3.9x4.9mm_Pitch0.635mm
- renumbered C42 to C56, C43 to C57, C44 to C58, C45 to C59, C46 to C64, C47 to C65, J4 to J2, J5 to J3
Connections:
- net RX1 is gone; now on net IN_CTS: IC1.12 (R1_O)
- net TX1 is gone; now on net IN_RTS: IC1.11 (T1_I)
- net +3V3: now also C60.1, C61.1, IC2.16 (VCC)
- net GND: now also C60.2, C61.2, C66.1, C67.1, IC2.15 (GND)
- net IN_RTS: now reaches J2.7 (P7)
- net IN_RTS: now also IC1.14 (T1_O)
- net IN_CTS: now reaches J2.8 (P8)
- net IN_CTS: now also IC1.13 (R1_I)
- net OUT_RTS: now reaches J3.7 (P7)
- net OUT_RTS: now also IC2.11 (T1_I), IC2.14 (T1_O)
- net OUT_CTS: now reaches J3.8 (P8)
- net OUT_CTS: now also IC2.12 (R1_O), IC2.13 (R1_I)
- net R1 renamed IN_RXD
- net IN_RXD: now also IC1.8 (R2_I); no longer IC1.13 (R1_I)
- net R2 renamed OUT_RXD
- net OUT_RXD: now also IC2.8 (R2_I); no longer IC1.8 (R2_I)
- net RX2 renamed IN_RX
- net T1 renamed IN_TXD
- net IN_TXD: now also IC1.7 (T2_O); no longer IC1.14 (T1_O)
- net T2 renamed OUT_TXD
- net OUT_TXD: now also IC2.7 (T2_O); no longer IC1.7 (T2_O)
- net TX2 renamed IN_TX
- new net: C62.1, IC2.1 (C1+)
- new net: C66.2, IC2.2 (V+)
- new net: C62.2, IC2.3 (C1-)
- new net: C63.1, IC2.4 (C2+)
- new net: C63.2, IC2.5 (C2-)
- new net: C67.2, IC2.6 (V-)
- new net OUT_RX: IC2.9 (R2_O)
- new net OUT_TX: IC2.10 (T2_I)
- no-connect marks 0 -> 8
Other:
- note added: "De verificat semnalele!!"
- note removed: "1 -> IN\n2 -> OUT"
- note removed: "CTS/RTS si restul semnalelor ?"
- note removed: "Liniile de TD si RD differential ?"
- note removed: "Power input ? ->"
- moved on the sheet: C56, C57, C58, C59, C64, C65, IC1, J2, J3
