File: SERIAL_RS232_conv.sch (KiCad schematic (older format))
At the start: 16 parts, among them IC1 MAX3232, IC2 MAX3232, J2 MDB9_IN, J3 MDB9_OUT

Commit message: Modified board. v1.1 to reflect the schematic change.
Connections:
- net IN_CTS: no longer IC1.13 (R1_I), J2.8 (P8)
- net IN_RTS: no longer IC1.14 (T1_O), J2.7 (P7)
- net OUT_CTS: no longer IC2.13 (R1_I), J3.8 (P8)
- net OUT_RTS: no longer IC2.14 (T1_O), J3.7 (P7)
- net IN_RXD renamed IN_RS_RXD
- net IN_TXD renamed IN_RS_TXD
- net OUT_RXD renamed OUT_RS_RXD
- net OUT_TXD renamed OUT_RS_TXD
- new net IN_RS_CTS: IC1.13 (R1_I), J2.8 (P8)
- new net IN_RS_RTS: IC1.14 (T1_O), J2.7 (P7)
- new net OUT_RS_CTS: IC2.13 (R1_I), J3.8 (P8)
- new net OUT_RS_RTS: IC2.14 (T1_O), J3.7 (P7)
Other:
- moved on the sheet: J3
Changed lines of the file:
@@
 L DB9 J3
 U 1 1 588F1F2B
-P 6100 3900
-F 0 "J3" H 6100 4450 50  0000 C CNN
-F 1 "MDB9_OUT" H 6100 3350 50  0000 C CNN
-F 2 "Connectors:DB9FC" H 6100 3900 50  0001 C CNN
-F 3 "" H 6100 3900 50  0000 C CNN
-	1    6100 3900
+P 6300 3800
+F 0 "J3" H 6300 4350 50  0000 C CNN
+F 1 "MDB9_OUT" H 6300 3250 50  0000 C CNN
+F 2 "Connectors:DB9FC" H 6300 3800 50  0001 C CNN
+F 3 "" H 6300 3800 50  0000 C CNN
+	1    6300 3800
 	1    0    0    -1
 $EndComp
 $Comp
-L GND #PWR099
+L GND #PWR0115
 U 1 1 588F1FE7
 P 5550 1700
-F 0 "#PWR099" H 5550 1450 50  0001 C CNN
+F 0 "#PWR0115" H 5550 1450 50  0001 C CNN
 F 1 "GND" H 5550 1550 50  0000 C CNN
 F 2 "" H 5550 1700 50  0000 C CNN
@@
 $EndComp
 $Comp
-L GND #PWR0100
+L GND #PWR0116
 U 1 1 588F2002
-P 5550 3500
-F 0 "#PWR0100" H 5550 3250 50  0001 C CNN
-F 1 "GND" H 5550 3350 50  0000 C CNN
-F 2 "" H 5550 3500 50  0000 C CNN
-F 3 "" H 5550 3500 50  0000 C CNN
-	1    5550 3500
+P 5750 3400
+F 0 "#PWR0116" H 5750 3150 50  0001 C CNN
+F 1 "GND" H 5750 3250 50  0000 C CNN
+F 2 "" H 5750 3400 50  0000 C CNN
+F 3 "" H 5750 3400 50  0000 C CNN
+	1    5750 3400
 	0    1    1    0
 $EndComp
@@
 	2100 2800 2600 2800
 $Comp
-L GND #PWR0101
+L GND #PWR0117
 U 1 1 588F251A
 P 4100 1800
-F 0 "#PWR0101" H 4100 1550 50  0001 C CNN
+F 0 "#PWR0117" H 4100 1550 50  0001 C CNN
 F 1 "GND" H 4100 1650 50  0000 C CNN
 F 2 "" H 4100 1800 50  0000 C CNN
@@
 Connection ~ 4050 1800
 $Comp
-L GND #PWR0102
+L GND #PWR0118
 U 1 1 588F266A
 P 2050 2000
-F 0 "#PWR0102" H 2050 1750 50  0001 C CNN
+F 0 "#PWR0118" H 2050 1750 50  0001 C CNN
 F 1 "GND" H 2050 1850 50  0000 C CNN
 F 2 "" H 2050 2000 50  0000 C CNN
@@
 Connection ~ 2100 2000
 $Comp
-L +3.3V #PWR0103
+L +3.3V #PWR0119
 U 1 1 588F26E1
 P 2550 1550
-F 0 "#PWR0103" H 2550 1400 50  0001 C CNN
+F 0 "#PWR0119" H 2550 1400 50  0001 C CNN
 F 1 "+3.3V" H 2550 1690 50  0000 C CNN
 F 2 "" H 2550 1550 50  0000 C CNN
@@
 	5550 1700 5650 1700
 Wire Wire Line
-	5550 3500 5650 3500
-Wire Wire Line
-	3600 2500 3700 2500
-Wire Wire Line
-	3600 2600 3700 2600
-Wire Wire Line
-	3600 2700 3700 2700
-Wire Wire Line
-	3600 2800 3700 2800
+	5750 3400 5850 3400
 Wire Wire Line
 	3600 1800 3650 1800
@@
 Wire Wire Line
 	3600 1900 3700 1900
-Wire Wire Line
-	3600 2050 3700 2050
-Wire Wire Line
-	3600 2150 3700 2150
-Wire Wire Line
-	3600 2250 3700 2250
-Wire Wire Line
-	3600 2350 3700 2350
 $Comp
 L MAX3232 IC2
@@
 	2150 4550 2650 4550
 $Comp
-L GND #PWR0104
+L GND #PWR0120
 U 1 1 58BE9045
 P 4150 3550
-F 0 "#PWR0104" H 4150 3300 50  0001 C CNN
+F 0 "#PWR0120" H 4150 3300 50  0001 C CNN
 F 1 "GND" H 4150 3400 50  0000 C CNN
 F 2 "" H 4150 3550 50  0000 C CNN
@@
 Connection ~ 4100 3550
 $Comp
-L GND #PWR0105
+L GND #PWR0121
 U 1 1 58BE9050
 P 2100 3750
-F 0 "#PWR0105" H 2100 3500 50  0001 C CNN
+F 0 "#PWR0121" H 2100 3500 50  0001 C CNN
 F 1 "GND" H 2100 3600 50  0000 C CNN
 F 2 "" H 2100 3750 50  0000 C CNN
@@
 Connection ~ 2150 3750
 $Comp
-L +3.3V #PWR0106
+L +3.3V #PWR0122
 U 1 1 58BE9057
 P 2600 3300
-F 0 "#PWR0106" H 2600 3150 50  0001 C CNN
+F 0 "#PWR0122" H 2600 3150 50  0001 C CNN
 F 1 "+3.3V" H 2600 3440 50  0000 C CNN
 F 2 "" H 2600 3300 50  0000 C CNN
@@
 	3650 4100 3750 4100
 Text Label 3700 2050 0    50   ~ 0
-IN_TXD
-Wire Wire Line
-	5550 2000 5650 2000
-Wire Wire Line
-	5550 2100 5650 2100
-Wire Wire Line
-	5550 2200 5650 2200
-Wire Wire Line
-	5550 2300 5650 2300
+IN_RS_TXD
 Text Label 3700 2350 0    50   ~ 0
-IN_CTS
+IN_RS_CTS
 Text Label 3700 2150 0    50   ~ 0
-IN_RTS
+IN_RS_RTS
 Text Label 3700 2250 0    50   ~ 0
-IN_RXD
+IN_RS_RXD
 Text HLabel 3700 2500 2    50   Output ~ 0
 IN_TX
@@
 IN_RTS
 Text Label 5550 2100 2    50   ~ 0
-IN_TXD
+IN_RS_TXD
 Text Label 5550 2000 2    50   ~ 0
-IN_CTS
+IN_RS_CTS
 Text Label 5550 2200 2    50   ~ 0
-IN_RTS
+IN_RS_RTS
 Text Label 5550 2300 2    50   ~ 0
-IN_RXD
+IN_RS_RXD
 Text Notes 4100 2200 0    50   ~ 0
 De verificat semnalele!!
 Text Label 3750 3800 0    50   ~ 0
-OUT_TXD
+OUT_RS_TXD
 Text Label 3750 3900 0    50   ~ 0
-OUT_RTS
+OUT_RS_RTS
 Text Label 3750 4000 0    50   ~ 0
-OUT_RXD
+OUT_RS_RXD
 Text Label 3750 4100 0    50   ~ 0
-OUT_CTS
-Text Label 5550 3800 2    50   ~ 0
-OUT_CTS
-Text Label 5550 3900 2    50   ~ 0
-OUT_TXD
-Text Label 5550 4000 2    50   ~ 0
-OUT_RTS
-Text Label 5550 4100 2    50   ~ 0
-OUT_RXD
-Wire Wire Line
-	5550 3800 5650 3800
-Wire Wire Line
-	5550 3900 5650 3900
-Wire Wire Line
-	5550 4000 5650 4000
-Wire Wire Line
-	5550 4100 5650 4100
-NoConn ~ 5650 3600
-NoConn ~ 5650 3700
-NoConn ~ 5650 4200
-NoConn ~ 5650 4300
+OUT_RS_CTS
+Text Label 5750 3700 2    50   ~ 0
+OUT_RS_CTS
+Text Label 5750 3800 2    50   ~ 0
+OUT_RS_TXD
+Text Label 5750 3900 2    50   ~ 0
+OUT_RS_RTS
+Text Label 5750 4000 2    50   ~ 0
+OUT_RS_RXD
+Wire Wire Line
+	5750 3700 5850 3700
+Wire Wire Line
+	5750 3800 5850 3800
+Wire Wire Line
+	5750 3900 5850 3900
+Wire Wire Line
+	5750 4000 5850 4000
+NoConn ~ 5850 3500
+NoConn ~ 5850 3600
+NoConn ~ 5850 4100
+NoConn ~ 5850 4200
 NoConn ~ 5650 1800
 NoConn ~ 5650 1900
@@
 Text HLabel 3750 4550 2    50   Input ~ 0
 OUT_CTS
-Text Notes 4200 3900 0    50   ~ 0
+Text Notes 4250 3900 0    50   ~ 0
 De verificat semnalele!!
+Wire Wire Line
+	3600 2050 3700 2050
+Wire Wire Line
+	3600 2150 3700 2150
+Wire Wire Line
+	3600 2250 3700 2250
+Wire Wire Line
+	3600 2350 3700 2350
+Wire Wire Line
+	5550 2000 5650 2000
+Wire Wire Line
+	5550 2100 5650 2100
+Wire Wire Line
+	5550 2200 5650 2200
+Wire Wire Line
+	5550 2300 5650 2300
+Wire Wire Line
+	3600 2500 3700 2500
+Wire Wire Line
+	3600 2600 3700 2600
+Wire Wire Line
+	3600 2700 3700 2700
+Wire Wire Line
+	3600 2800 3700 2800
 $EndSCHEMATC
