File: E-GIF-M-Board.kicad_pcb (KiCad board)
At the start: 2 copper layers, 100 x 100 mm, 133 parts, among them CON1 PWR_JACK, CON2 Micro_SD_Card, CON3 RJ45-TRF-LED, CON4 RJ45-TRF-LED, IC1 MAX3232, J4 MDB9_IN, J5 MDB9_OUT, P4 DEBUG, P6 TB_IN, P7 TB_OUT, U1 MCP16312-E/MS, U2 ARIA-G25, U3 MCP2200, U4 LAN9500A, U5 ST3485EBDR, U6 ST3485EBDR, Y1 16MHz, Y2 25MHz

Commit message: Modified schematic. v1.1
Parts:
- removed P4: DEBUG, Custom:MicroUSB-B
- removed P6: TB_IN, Connectors_Terminal_Blocks:TerminalBlock_Pheonix_PT-3.5mm_2pol
- removed P7: TB_OUT, Connectors_Terminal_Blocks:TerminalBlock_Pheonix_PT-3.5mm_2pol
- removed REF** (x26): SolderWirePad_single_0-8mmDrill, Wire_Pads:SolderWirePad_single_0-8mmDrill
- removed S1: ~RST, misc:SW_SPST_EVPBF
- added C48: .022uF, Capacitors_Tantalum_SMD:CP_Tantalum_Case-C_EIA-6032-28_Hand, F.Cu at (183.3, 113.0)
- added C49, C56, C60, C69, C71, C72: 100nF, Capacitors_SMD:C_0603_HandSoldering, F.Cu at (183.3, 113.0)
- added C52, C53, C57, C58, C59, C61, C62, C63, C64, C65, C66, C67: 0.1uF, Capacitors_SMD:C_0603_HandSoldering, F.Cu at (183.3, 113.0)
- added C68, C70: 1uF, Capacitors_SMD:C_0603_HandSoldering, F.Cu at (183.3, 113.0)
- added D10, D11, D12, D13, D14, D15: D_TVS, Diodes_SMD:D_SMA-SMB_Universal_Handsoldering, F.Cu at (183.3, 113.0)
- added D7, D8: LED, LEDs:LED_0603, F.Cu at (183.3, 113.0)
- added D9: FDX_LED, LEDs:LED_0603, F.Cu at (183.3, 113.0)
- added IC2: MAX3232, Housings_SSOP:SSOP-16_3.9x4.9mm_Pitch0.635mm, F.Cu at (183.3, 113.0)
- added J1: 1W_H, Pin_Headers:Pin_Header_Straight_1x02_Pitch1.27mm, F.Cu at (183.3, 113.0)
- added J2: MDB9_IN, Connectors:DB9FC, F.Cu at (214.7, 149.5)
- added J3: MDB9_OUT, Connectors:DB9FC, F.Cu at (179.1, 155.5)
- added JP1, JP2, JP3, JP4, JP5, JP6: Jumper_NO_Small, Pin_Headers:Pin_Header_Straight_1x02_Pitch2.54mm, F.Cu at (183.3, 113.0)
- added P1: USB_A, Connect:USB_A, F.Cu at (147.8, 113.0)
- added P2: DEBUG, Custom:MicroUSB-B, F.Cu at (183.3, 113.0)
- added R21, R42: 10k, Resistors_SMD:R_0603_HandSoldering, F.Cu at (183.3, 113.0)
- added R22, R25, R34: 1M, Resistors_SMD:R_0603_HandSoldering, F.Cu at (183.3, 113.0)
- added R23, R24: 220, Resistors_SMD:R_0603_HandSoldering, F.Cu at (183.3, 113.0)
- added R26, R29, R30, R31: 49.9, Resistors_SMD:R_0603_HandSoldering, F.Cu at (183.3, 113.0)
- added R27, R28: 12k, Resistors_SMD:R_0603_HandSoldering, F.Cu at (183.3, 113.0)
- added R32, R33, R35: 330, Resistors_SMD:R_0603_HandSoldering, F.Cu at (183.3, 113.0)
- added R36, R37, R38, R39, R40, R41: R, Resistors_SMD:R_0603_HandSoldering, F.Cu at (183.3, 113.0)
- added SW1: BTN, Buttons_Switches_SMD:SW_SPST_EVQPE1, F.Cu at (183.3, 113.0)
- added SW2: ~RST, Buttons_Switches_SMD:SW_SPST_EVQPE1, F.Cu at (183.3, 113.0)
- added U7: ST3485EBDR, Power_Integrations:SO-8, F.Cu at (183.3, 113.0)
- added W10: RXD2_T, Measurement_Points:Measurement_Point_Round-SMD-Pad_Small, F.Cu at (183.3, 113.0)
- added W11: TXD3_T, Measurement_Points:Measurement_Point_Round-SMD-Pad_Small, F.Cu at (183.3, 113.0)
- added W12: RXD3_T, Measurement_Points:Measurement_Point_Round-SMD-Pad_Small, F.Cu at (183.3, 113.0)
- added W13: DRXD_T, Measurement_Points:Measurement_Point_Round-SMD-Pad_Small, F.Cu at (183.3, 113.0)
- added W14: DTXD_T, Measurement_Points:Measurement_Point_Round-SMD-Pad_Small, F.Cu at (183.3, 113.0)
- added W15: U2S_RST, Measurement_Points:Measurement_Point_Round-SMD-Pad_Small, F.Cu at (183.3, 113.0)
- added W16: U2E_RST, Measurement_Points:Measurement_Point_Round-SMD-Pad_Small, F.Cu at (183.3, 113.0)
- added W6: RXD0_T, Measurement_Points:Measurement_Point_Round-SMD-Pad_Small, F.Cu at (183.3, 113.0)
- added W7: TXD1_T, Measurement_Points:Measurement_Point_Round-SMD-Pad_Small, F.Cu at (183.3, 113.0)
- added W8: RXD1_T, Measurement_Points:Measurement_Point_Round-SMD-Pad_Small, F.Cu at (183.3, 113.0)
- added W9: TXD2_T, Measurement_Points:Measurement_Point_Round-SMD-Pad_Small, F.Cu at (183.3, 113.0)
- C1, C2, C5, C6: footprint Capacitors_SMD:C_0603_HandSoldering -> Capacitors_Tantalum_SMD:CP_Tantalum_Case-C_EIA-6032-28_Hand
- C10, C22: value 1uF -> 100nF
- C11, C12, C14: value 1uF -> 10uF
- C13: value 100nF -> 10uF
- C23: value 6pF -> 1uF
- C24: value 6pF -> 100nF
- C25, C27, C32: value 0.1uF -> 100nF
- C26: value 0.1uF -> 10uF
- C28, C33: value 0.1uF -> 1uF
- C29: value 0.1uF -> 1nF; moved to F.Cu
- C3: value 1uF -> 10uF; footprint Capacitors_SMD:C_0603_HandSoldering -> Capacitors_Tantalum_SMD:CP_Tantalum_Case-C_EIA-6032-28_Hand
- C30, C31: value 0.1uF -> 1nF
- C34: value .022uF -> 6pF
- C35: value 22pF -> 6pF
- C36: value 22pF -> 1nF
- C4: value 100nF -> 10uF; footprint Capacitors_SMD:C_0603_HandSoldering -> Capacitors_Tantalum_SMD:CP_Tantalum_Case-C_EIA-6032-28_Hand
- C42, C55: value 100nF -> 0.1uF
- C46, C47: value 0.1uF -> 22pF
- C50, C54: value 1uF -> 0.1uF
- C7, C8: value 100nF -> 1uF
- CON2: value Micro_SD_Card -> RJ45-TRF-LED; footprint Custom:MicroSDSocket -> misc:RJ45_TRANSFO; moved to F.Cu
- CON3: value RJ45-TRF-LED -> Micro_SD_Card; footprint misc:RJ45_TRANSFO -> Custom:MicroSDSocket
- D1, D2: footprint Diodes_SMD:D_SMA_Handsoldering -> Diodes_SMD:D_SMA-SMB_Universal_Handsoldering
- D4: value LED -> PWR_LED
- D6: value FDX_LED -> TL431DBZ; footprint LEDs:LED_0603 -> TO_SOT_Packages_SMD:SOT-23
- IC1: footprint SMD_Packages:SO-16-L -> Housings_SSOP:SSOP-16_3.9x4.9mm_Pitch0.635mm
- J4: value MDB9_IN -> Screw_Terminal_1x03; footprint Connectors:DB9FC -> Connectors_Terminal_Blocks:TerminalBlock_Pheonix_PT-3.5mm_3pol
- J5: value MDB9_OUT -> Screw_Terminal_1x03; footprint Connectors:DB9FC -> Connectors_Terminal_Blocks:TerminalBlock_Pheonix_PT-3.5mm_3pol
- L2: value LF -> 22uH; footprint Resistors_SMD:R_0603_HandSoldering -> Inductors:Inductor_Taiyo-Yuden_MD-5050
- R1: value 31k6 -> 1M
- R10, R6: value 49.9 -> 10k
- R11, R9: value 49.9 -> R
- R12, R13, R14: value 330 -> R
- R15, R16, R18: value 1M -> R
- R17: value 1k -> R
- R2: value 10k -> 1M
- R3: value 220 -> 31k6
- R4: value 220 -> 10k
- R5: value 220 -> 52k3
- R7, R8: value 12k -> 220
- U1: footprint Housings_SSOP:MSOP-8-1EP_3x3mm_Pitch0.65mm -> Housings_SSOP:MSOP-8_3x3mm_Pitch0.65mm
- U2: value ARIA-G25 -> MCP16312-E/MS; footprint misc:ARIA-G25 -> Housings_SSOP:MSOP-8_3x3mm_Pitch0.65mm
- U3: value MCP2200 -> ARIA-G25; footprint Housings_SSOP:SSOP-20_5.3x7.2mm_Pitch0.65mm -> misc:ARIA-G25
- U4: value LAN9500A -> MCP2200; footprint Housings_DFN_QFN:QFN-56-1EP_7x7mm_Pitch0.4mm -> Housings_SSOP:SSOP-20_4.4x6.5mm_Pitch0.65mm
- U5: value ST3485EBDR -> LAN9500A; footprint Power_Integrations:SO-8 -> Housings_DFN_QFN:QFN-56-1EP_7x7mm_Pitch0.4mm
- W1: value 3.3V_T -> VBUS_T; footprint Measurement_Points:Measurement_Point_Square-SMD-Pad_Small -> Measurement_Points:Measurement_Point_Round-SMD-Pad_Small
- W2: value U2S_RST -> VIN_T
- W3: value RX_T -> 3.3V_T; footprint Pin_Headers:Pin_Header_Straight_1x01_Pitch2.54mm -> Measurement_Points:Measurement_Point_Round-SMD-Pad_Small
- W4: value TX_T -> 5V_T; footprint Pin_Headers:Pin_Header_Straight_1x01_Pitch2.54mm -> Measurement_Points:Measurement_Point_Round-SMD-Pad_Small
- W5: value U2E_RST -> TXD0_T
- moved C15 179.3 mm to (216.8, 68.7)
- moved C44 179.3 mm to (251.7, 54.3)
- moved IC1 179.3 mm to (239.2, 58.7)
- moved C11 179.3 mm to (242.2, 88.2)
- moved C12 179.3 mm to (220.2, 49.9)
- moved C13 179.3 mm to (217.8, 52.2)
- moved C14 179.3 mm to (220.2, 45.9)
- moved C16 179.3 mm to (215.1, 71.0)
- moved C42 179.3 mm to (235.4, 52.4)
- moved C43 179.3 mm to (235.4, 50.2)
- moved C45 179.3 mm to (251.8, 58.1)
- moved C46 179.3 mm to (248.1, 54.3)
- moved C47 179.3 mm to (251.8, 60.7)
- moved C9 179.3 mm to (220.2, 47.9)
- moved CON3 179.3 mm to (215.2, 86.1)
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Connections:
- C1 pad 1: /Power/VIN -> /VIN
- C10 pad 1: +3V3 -> Net-(C10-Pad1)
- C10 pad 2: GND -> Net-(C10-Pad2)
- C11 pad 1: /AriaG25Module/~RST -> +3V3
- C12 pad 1: +3V3 -> +5V
- C14 pad 1: +3V3 -> +5V
- C2 pad 1: /Power/VIN -> /VIN
- C22 pad 1: +3V3 -> GND
- C22 pad 2: GND -> Net-(C22-Pad2)
- C23 pad 1: GND -> +3V3
- C23 pad 2: /Interfaces/OSC2 -> GND
- C24 pad 2: /Interfaces/OSC1 -> Net-(C24-Pad2)
- C25 pad 1: +3V3 -> /AriaG25Module/~RST
- C29 pad 1: +3V3 -> GND
- C29 pad 2: GND -> Net-(C29-Pad2)
- C3 pad 1: Net-(C3-Pad1) -> /VIN
- C30 pad 1: /Interfaces/USB_ETH_conv/VDD33A -> GND
- C30 pad 2: GND -> Net-(C30-Pad2)
- C31 pad 1: /Interfaces/USB_ETH_conv/VDD33A -> GND
- C31 pad 2: GND -> Net-(C31-Pad2)
- C32 pad 1: /Interfaces/USB_ETH_conv/VDD33A -> +3V3
- C33 pad 1: /Interfaces/USB_ETH_conv/VDD33A -> +3V3
- C34 pad 1: /Interfaces/USB_ETH_conv/VDD33A -> GND
- C34 pad 2: GND -> /Interfaces/OSC2
- C35 pad 1: Net-(C35-Pad1) -> GND
- C35 pad 2: GND -> /Interfaces/OSC1
- C36 pad 1: Net-(C36-Pad1) -> GND
- C36 pad 2: GND -> Net-(C36-Pad2)
- C37 pad 1: /Interfaces/USB_ETH_conv/VDDUSBPLL -> +3V3
- C38 pad 1: /Interfaces/USB_ETH_conv/VDDCORE -> +3V3
- C39 pad 1: /Interfaces/USB_ETH_conv/VDDCORE -> +3V3
- C4 pad 1: Net-(C4-Pad1) -> /VIN
- C4 pad 2: Net-(C4-Pad2) -> GND
- C40 pad 1: /Interfaces/USB_ETH_conv/VDDCORE -> +3V3
- C41 pad 1: /Interfaces/USB_ETH_conv/VDDPLL -> +3V3
- C42 pad 1: +3V3 -> /Interfaces/USB_ETH_conv/VDD33A
- C43 pad 1: +3V3 -> /Interfaces/USB_ETH_conv/VDD33A
- C44 pad 1: Net-(C44-Pad1) -> /Interfaces/USB_ETH_conv/VDD33A
- C44 pad 2: Net-(C44-Pad2) -> GND
- C45 pad 1: Net-(C45-Pad1) -> /Interfaces/USB_ETH_conv/VDD33A
- C45 pad 2: Net-(C45-Pad2) -> GND
- C46 pad 1: GND -> Net-(C46-Pad1)
- C46 pad 2: Net-(C46-Pad2) -> GND
- C47 pad 1: GND -> Net-(C47-Pad1)
- C47 pad 2: Net-(C47-Pad2) -> GND
- C5 pad 1: +3V3 -> /VIN
- C50 pad 1: GND -> /Interfaces/USB_ETH_conv/VDDUSBPLL
- C50 pad 2: +3V3 -> GND
- C51 pad 2: +3V3 -> Net-(C51-Pad2)
- C54 pad 1: GND -> /Interfaces/USB_ETH_conv/VDDCORE
- C54 pad 2: +3V3 -> GND
- C55 pad 1: GND -> /Interfaces/USB_ETH_conv/VDDPLL
- C55 pad 2: +3V3 -> GND
- C6 pad 1: +3V3 -> /VIN
- C7 pad 1: +3V3 -> Net-(C7-Pad1)
- C8 pad 1: /AriaG25Module/~RST -> Net-(C8-Pad1)
- C9 pad 1: +3V3 -> Net-(C9-Pad1)
- C9 pad 2: GND -> Net-(C9-Pad2)
- CON2 pad 1: /AriaG25Module/DA2 -> /AriaG25Module/ETHTX_P
- CON2 pad 10: (no net) -> GND
- CON2 pad 2: /AriaG25Module/DA3 -> /AriaG25Module/ETHTX_N
- CON2 pad 3: /AriaG25Module/CDA -> /AriaG25Module/ETH3V3
- CON2 pad 4: +3V3 -> Net-(C29-Pad2)
- CON2 pad 5: /AriaG25Module/CK -> Net-(C29-Pad2)
- CON2 pad 6: GND -> /AriaG25Module/ETH3V3
- CON2 pad 7: /AriaG25Module/DA0 -> /AriaG25Module/ETHRX_P
- CON2 pad 8: /AriaG25Module/DA1 -> /AriaG25Module/ETHRX_N
- CON2 pad 9: Net-(CON2-Pad9) -> /AriaG25Module/ETHLED1
- CON3 pad 1: /AriaG25Module/ETHRX_P -> /AriaG25Module/DA2
- CON3 pad 2: +3V3 -> /AriaG25Module/DA3
- CON3 pad 3: /AriaG25Module/ETHRX_N -> /AriaG25Module/CDA
- CON3 pad 4: Net-(CON3-Pad4) -> +3V3
- CON3 pad 5: Net-(CON3-Pad4) -> /AriaG25Module/CK
- CON3 pad 6: +3V3 -> GND
- CON3 pad 7: /AriaG25Module/ETHTX_P -> /AriaG25Module/DA0
- CON3 pad 8: /AriaG25Module/ETHTX_N -> /AriaG25Module/DA1
- CON3 pad 9: /AriaG25Module/ETHLED1 -> Net-(C30-Pad2)
- CON4 pad 4: Net-(CON4-Pad4) -> Net-(C51-Pad2)
- CON4 pad 5: Net-(CON4-Pad4) -> Net-(C51-Pad2)
- D1 pad 1: /Power/VIN -> /VIN
- D2 pad 1: /Power/VIN -> /VIN
- D4 pad 1: GND -> Net-(D4-Pad1)
- D4 pad 2: Net-(D4-Pad2) -> +5V
- D6 pad 1: Net-(D6-Pad1) -> +3V3
- IC1 pad 1: Net-(C44-Pad1) -> Net-(C58-Pad1)
- IC1 pad 10: /Interfaces/RS232_OUT_TX -> /Interfaces/RS232_IN_TX
- IC1 pad 11: /Interfaces/RS232_IN_TX -> /Interfaces/RS232_IN_RTS
- IC1 pad 12: /Interfaces/RS232_IN_RX -> /AriaG25Module/CTS0
- IC1 pad 13: /Interfaces/SERIAL_RS232_conv/R1 -> /AriaG25Module/CTS0
- IC1 pad 14: /Interfaces/SERIAL_RS232_conv/T1 -> /Interfaces/RS232_IN_RTS
- IC1 pad 2: Net-(C46-Pad2) -> Net-(C64-Pad2)
- IC1 pad 3: Net-(C44-Pad2) -> Net-(C58-Pad2)
- IC1 pad 4: Net-(C45-Pad1) -> Net-(C59-Pad1)
- IC1 pad 5: Net-(C45-Pad2) -> Net-(C59-Pad2)
- IC1 pad 6: Net-(C47-Pad2) -> Net-(C65-Pad2)
- IC1 pad 7: /Interfaces/SERIAL_RS232_conv/T2 -> /Interfaces/SERIAL_RS232_conv/IN_TXD
- IC1 pad 8: /Interfaces/SERIAL_RS232_conv/R2 -> /Interfaces/SERIAL_RS232_conv/IN_RXD
- IC1 pad 9: /Interfaces/RS232_OUT_RX -> /Interfaces/RS232_IN_RX
- J4 pad 1: Net-(J4-Pad1) -> GND
- J4 pad 2: /Interfaces/SERIAL_RS232_conv/R1 -> Net-(D11-Pad2)
- J4 pad 3: /Interfaces/SERIAL_RS232_conv/T1 -> Net-(D10-Pad2)
- J5 pad 1: Net-(J5-Pad1) -> GND
- J5 pad 2: /Interfaces/SERIAL_RS232_conv/R2 -> Net-(D14-Pad2)
- J5 pad 3: /Interfaces/SERIAL_RS232_conv/T2 -> Net-(D13-Pad2)
- L1 pad 2: Net-(C4-Pad1) -> Net-(C9-Pad1)
- L2 pad 1: +3V3 -> +5V
- L2 pad 2: /AriaG25Module/ADVREF -> Net-(C10-Pad1)
- R1 pad 1: +3V3 -> Net-(R1-Pad1)
- R1 pad 2: /Power/VFB -> /VIN
- R10 pad 1: /Interfaces/USB_ETH_conv/VDD33A -> +3V3
- R10 pad 2: /Interfaces/USB_ETH_conv/TX+ -> /AriaG25Module/~RST
- R11 pad 1: /Interfaces/USB_ETH_conv/VDD33A -> +3V3
- R11 pad 2: /Interfaces/USB_ETH_conv/TX- -> /AriaG25Module/3V3_DIV
- R12 pad 1: /Interfaces/USB_ETH_conv/nLNKA_LED -> /AriaG25Module/3V3_DIV
- R12 pad 2: Net-(CON4-Pad10) -> GND
- R13 pad 1: /Interfaces/USB_ETH_conv/nSPD_LED -> +5V
- R13 pad 2: Net-(CON4-Pad12) -> /AriaG25Module/5V_DIV
- R14 pad 1: Net-(D6-Pad1) -> /AriaG25Module/5V_DIV
- R14 pad 2: /Interfaces/USB_ETH_conv/nFDX_LED -> GND
- R15 pad 1: Net-(CON3-Pad4) -> /VBUS
- R15 pad 2: GND -> /AriaG25Module/VBUS_DIV
- R16 pad 1: GND -> /AriaG25Module/VBUS_DIV
- R16 pad 2: Net-(CON2-Pad9) -> GND
- R17 pad 1: +3V3 -> /VIN
- R17 pad 2: /AriaG25Module/~RST -> /AriaG25Module/VIN_DIV
- R18 pad 1: Net-(R18-Pad1) -> /AriaG25Module/VIN_DIV
- R18 pad 2: /Power/VIN -> GND
- R19 pad 1: Net-(P4-Pad6) -> Net-(C29-Pad2)
- R2 pad 1: /Power/VFB -> Net-(R2-Pad1)
- R2 pad 2: GND -> /VIN
- R20 pad 2: Net-(CON4-Pad4) -> Net-(C30-Pad2)
- R3 pad 1: GND -> +3V3
- R3 pad 2: Net-(D3-Pad1) -> /Power/3V3_VFB
- R4 pad 1: Net-(R4-Pad1) -> /Power/3V3_VFB
- R4 pad 2: Net-(D4-Pad2) -> GND
- R5 pad 1: Net-(R5-Pad1) -> +5V
- R5 pad 2: Net-(D5-Pad2) -> /Power/5V_VFB
- R6 pad 1: /Interfaces/USB_ETH_conv/VDD33A -> /Power/5V_VFB
- R6 pad 2: /Interfaces/USB_ETH_conv/RX+ -> GND
- R7 pad 2: Net-(R7-Pad2) -> Net-(D3-Pad1)
- R8 pad 2: Net-(R8-Pad2) -> Net-(D4-Pad1)
- R9 pad 1: /Interfaces/USB_ETH_conv/VDD33A -> Net-(R9-Pad1)
- R9 pad 2: /Interfaces/USB_ETH_conv/RX- -> Net-(D5-Pad2)
- U1 pad 1: /Power/VFB -> /Power/3V3_VFB
- U1 pad 2: Net-(C3-Pad1) -> Net-(C7-Pad1)
- U1 pad 3: Net-(R18-Pad1) -> Net-(R1-Pad1)
- U1 pad 4: /Power/VIN -> /VIN
- U1 pad 6: Net-(C4-Pad1) -> Net-(C9-Pad1)
- U1 pad 7: Net-(C4-Pad2) -> Net-(C9-Pad2)
- U4 pad 1: Net-(U4-Pad1) -> +3V3
- U4 pad 10: /Interfaces/USB_ETH_conv/VDDPLL -> /AriaG25Module/DRXD
- U4 pad 11: /AriaG25Module/USBA_N -> (no net)
- U4 pad 12: /AriaG25Module/USBA_P -> /AriaG25Module/DTXD
- U4 pad 13: GND -> (no net)
- U4 pad 14: Net-(U4-Pad14) -> (no net)
- U4 pad 15: /Interfaces/USB_ETH_conv/VDD33A -> (no net)
- U4 pad 16: Net-(R8-Pad2) -> (no net)
- U4 pad 17: /Interfaces/USB_ETH_conv/VDDUSBPLL -> +3V3
- U4 pad 18: Net-(C36-Pad1) -> /Interfaces/D-
- U4 pad 19: Net-(C35-Pad1) -> /Interfaces/D+
- U4 pad 2: /Interfaces/USB_ETH_conv/TX- -> /Interfaces/OSC1
- U4 pad 20: +3V3 -> GND
- U4 pad 3: /Interfaces/USB_ETH_conv/TX+ -> /Interfaces/OSC2
- U4 pad 4: /Interfaces/USB_ETH_conv/VDD33A -> Net-(C72-Pad1)
- U4 pad 5: /Interfaces/USB_ETH_conv/RX- -> Net-(R24-Pad1)
- U4 pad 6: /Interfaces/USB_ETH_conv/RX+ -> Net-(R23-Pad1)
- U4 pad 7: /Interfaces/USB_ETH_conv/VDD33A -> (no net)
- U4 pad 8: Net-(R7-Pad2) -> (no net)
- U4 pad 9: /Interfaces/USB_ETH_conv/VDD33A -> (no net)
- U5 pad 1: /Interfaces/RS485_IN_RO -> (no net)
- U5 pad 2: GND -> /Interfaces/USB_ETH_conv/TX-
- U5 pad 3: +3V3 -> /Interfaces/USB_ETH_conv/TX+
- U5 pad 4: /Interfaces/RS485_IN_DI -> /Interfaces/USB_ETH_conv/VDD33A
- U5 pad 5: GND -> /Interfaces/USB_ETH_conv/RX-
- U5 pad 6: Net-(P6-Pad1) -> /Interfaces/USB_ETH_conv/RX+
- U5 pad 7: Net-(P6-Pad2) -> /Interfaces/USB_ETH_conv/VDD33A
- U5 pad 8: +3V3 -> Net-(R27-Pad2)
- U6 pad 1: /Interfaces/RS485_OUT_RO -> /Interfaces/RS485_IN_RO
- U6 pad 2: GND -> /Interfaces/RS485_IN_RTS
- U6 pad 3: +3V3 -> /Interfaces/RS485_IN_RTS
- U6 pad 4: /Interfaces/RS485_OUT_DI -> /Interfaces/RS485_IN_DI
- U6 pad 6: Net-(P7-Pad1) -> Net-(D10-Pad2)
- U6 pad 7: Net-(P7-Pad2) -> Net-(D11-Pad2)
- W1 pad 1: +3V3 -> /VIN
- W2 pad 1: Net-(U3-Pad4) -> /VIN
- W3 pad 1: /AriaG25Module/DTXD -> +3V3
- W4 pad 1: /AriaG25Module/DRXD -> +5V
- W5 pad 1: /AriaG25Module/PC31 -> /Interfaces/RS232_IN_TX
- Y2 pad 1: Net-(C36-Pad1) -> Net-(C47-Pad1)
- Y2 pad 3: Net-(C35-Pad1) -> Net-(C46-Pad1)
Routing:
- net +3V3: track 451.1 -> 0.00 mm, vias 15 -> 0
- net /VBUS: track 116.6 -> 0.00 mm, vias 1 -> 0
- net /AriaG25Module/VBAT: track 71.6 -> 0.00 mm, vias 2 -> 0
- net /Interfaces/RS485_OUT_DI: track 66.4 -> 0.00 mm, vias 2 -> 0
- net /Interfaces/RS485_OUT_RO: track 60.9 -> 0.00 mm
- net /Interfaces/SERIAL_RS232_conv/R2: track 52.4 -> 0.00 mm, vias 1 -> 0
- net /AriaG25Module/~RST: track 52.4 -> 0.00 mm, vias 2 -> 0
- net /Interfaces/SERIAL_RS232_conv/T2: track 51.7 -> 0.00 mm, vias 1 -> 0
- net /Interfaces/USB_ETH_conv/VDD33A: track 44.7 -> 0.00 mm, vias 3 -> 0
- net /AriaG25Module/DTXD: track 43.0 -> 0.00 mm, vias 1 -> 0
- net /AriaG25Module/CDA: track 39.9 -> 0.00 mm, vias 3 -> 0
- net /AriaG25Module/DA2: track 36.7 -> 0.00 mm, vias 1 -> 0
- net /Interfaces/RS232_OUT_RX: track 36.0 -> 0.00 mm, vias 1 -> 0
- net /Interfaces/RS485_IN_RO: track 35.7 -> 0.00 mm
- net /AriaG25Module/DA1: track 35.6 -> 0.00 mm, vias 1 -> 0
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
Commit message: Modified board. v1.1 to reflect the schematic change.
Parts:
- added R43: R, Resistors_SMD:R_0603_HandSoldering, B.Cu at (53.3, 44.5)
- C1, C2, C3, C4, C5, C6: footprint Capacitors_Tantalum_SMD:CP_Tantalum_Case-C_EIA-6032-28_Hand -> Capacitors_Tantalum_SMD:CP_Tantalum_Case-B_EIA-3528-21_Hand
- C10, C11, C12, C13, C14, C17, C18, C22, C24, C29, C30, C37, C38, C49, C50, C52, C53, C54, C55, C7, C8, C9, CON3, D6, L2, L4, L5, P1, R12, R13, R14, R19, R20, R26, R29, R3, R30, R31, R32, R33, R4, R5, R6, U2: moved to B.Cu
- C25, C27, C33, C34, C35, C36, C46, C47, D1, D2, IC1, R10, R16, R18, R7, R8, R9, U4, Y2: moved to F.Cu
- W2: value VIN_T -> VJACK_T
- moved IC1 206.2 mm to (34.7, 85.2), turned to 90 degrees
- moved C11 199.5 mm to (51.1, 31.1), turned to 180 degrees
- moved J2 196.6 mm to (27.0, 90.9), turned to 90 degrees
- moved R18 196.5 mm to (37.6, 37.8), turned to 0 degrees
- moved L1 194.6 mm to (55.1, 39.7), turned to 0 degrees
- moved C5 191.8 mm to (66.0, 26.9), turned to 270 degrees
- moved W1 189.6 mm to (59.9, 115.5)
- moved R15 188.4 mm to (38.4, 34.7), turned to 180 degrees
- moved U1 185.7 mm to (55.2, 31.1), turned to 270 degrees
- moved R1 185.2 mm to (55.3, 24.6), turned to 0 degrees
- moved U2 178.9 mm to (66.3, 36.5)
- moved C4 176.1 mm to (72.0, 28.0), turned to 0 degrees
- moved R2 174.7 mm to (65.2, 32.2)
- moved C15 174.5 mm to (48.5, 22.9), turned to 0 degrees
- moved C16 173.8 mm to (48.5, 21.6), turned to 0 degrees
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Connections:
- net /Interfaces/SERIAL_RS232_conv/IN_RXD renamed /Interfaces/SERIAL_RS232_conv/IN_RS_RXD
- net /Interfaces/SERIAL_RS232_conv/IN_TXD renamed /Interfaces/SERIAL_RS232_conv/IN_RS_TXD
- net /Interfaces/SERIAL_RS232_conv/OUT_RXD renamed /Interfaces/SERIAL_RS232_conv/OUT_RS_RXD
- net /Interfaces/SERIAL_RS232_conv/OUT_TXD renamed /Interfaces/SERIAL_RS232_conv/OUT_RS_TXD
- C1 pad 1: /VIN -> /Power/VIN
- C2 pad 1: /VIN -> /Power/VIN
- C3 pad 1: /VIN -> /Power/VIN
- C4 pad 1: /VIN -> /Power/VIN
- C5 pad 1: /VIN -> /Power/VIN
- C6 pad 1: /VIN -> /Power/VIN
- CON1 pad 1: Net-(CON1-Pad1) -> /VJACK
- D1 pad 1: /VIN -> /Power/VIN
- D2 pad 1: /VIN -> /Power/VIN
- D2 pad 2: Net-(CON1-Pad1) -> /VJACK
- D6 pad 1: +3V3 -> /AriaG25Module/ADVREF
- D6 pad 2: +3V3 -> /AriaG25Module/ADVREF
- IC1 pad 13: /AriaG25Module/CTS0 -> /Interfaces/SERIAL_RS232_conv/IN_RS_CTS
- IC1 pad 14: /Interfaces/RS232_IN_RTS -> /Interfaces/SERIAL_RS232_conv/IN_RS_RTS
- IC2 pad 12: /AriaG25Module/CTS1 -> /AriaG25Module/CTS3
- IC2 pad 13: /AriaG25Module/CTS1 -> /Interfaces/SERIAL_RS232_conv/OUT_RS_CTS
- IC2 pad 14: /Interfaces/RS232_OUT_RTS -> /Interfaces/SERIAL_RS232_conv/OUT_RS_RTS
- J2 pad 1: (no net) -> Net-(J2-Pad1)
- J2 pad 4: (no net) -> Net-(J2-Pad4)
- J2 pad 6: (no net) -> Net-(J2-Pad6)
- J2 pad 7: /Interfaces/RS232_IN_RTS -> /Interfaces/SERIAL_RS232_conv/IN_RS_RTS
- J2 pad 8: /AriaG25Module/CTS0 -> /Interfaces/SERIAL_RS232_conv/IN_RS_CTS
- J2 pad 9: (no net) -> Net-(J2-Pad9)
- J3 pad 1: (no net) -> Net-(J3-Pad1)
- J3 pad 4: (no net) -> Net-(J3-Pad4)
- J3 pad 6: (no net) -> Net-(J3-Pad6)
- J3 pad 7: /Interfaces/RS232_OUT_RTS -> /Interfaces/SERIAL_RS232_conv/OUT_RS_RTS
- J3 pad 8: /AriaG25Module/CTS1 -> /Interfaces/SERIAL_RS232_conv/OUT_RS_CTS
- J3 pad 9: (no net) -> Net-(J3-Pad9)
- P2 pad 4: (no net) -> Net-(P2-Pad4)
- R1 pad 2: /VIN -> /Power/VIN
- R11 pad 1: +3V3 -> /5V_DIV
- R11 pad 2: /AriaG25Module/3V3_DIV -> GND
- R12 pad 1: /AriaG25Module/3V3_DIV -> +5V
- R12 pad 2: GND -> /5V_DIV
- R13 pad 1: +5V -> /3V3_DIV
- R13 pad 2: /AriaG25Module/5V_DIV -> GND
- R14 pad 1: /AriaG25Module/5V_DIV -> +3V3
- R14 pad 2: GND -> /3V3_DIV
- R15 pad 1: /VBUS -> /VJACK_DIV
- R15 pad 2: /AriaG25Module/VBUS_DIV -> GND
- R16 pad 1: /AriaG25Module/VBUS_DIV -> /VJACK
- R16 pad 2: GND -> /VJACK_DIV
- R17 pad 1: /VIN -> /VBUS_DIV
- R17 pad 2: /AriaG25Module/VIN_DIV -> GND
- R18 pad 1: /AriaG25Module/VIN_DIV -> /VBUS
- R18 pad 2: GND -> /VBUS_DIV
- R2 pad 2: /VIN -> /Power/VIN
- U1 pad 4: /VIN -> /Power/VIN
- U2 pad 4: /VIN -> /Power/VIN
- U3 pad E12: (no net) -> /AriaG25Module/USBC_P
- U3 pad E13: (no net) -> /AriaG25Module/USBC_N
- U3 pad E2: /Interfaces/RS485_IN_DI -> /Interfaces/RS232_OUT_TX
- U3 pad E3: /Interfaces/RS485_IN_RO -> /Interfaces/RS232_OUT_RX
- U3 pad E4: /Interfaces/RS485_IN_RTS -> /Interfaces/RS232_OUT_RTS
- U3 pad E5: (no net) -> /AriaG25Module/CTS3
- U3 pad E6: (no net) -> /AriaG25Module/PC26
- U3 pad E7: /Interfaces/RS232_OUT_RTS -> /Interfaces/RS485_OUT_RTS
- U3 pad E9: (no net) -> /AriaG25Module/PC29
- U3 pad N10: (no net) -> Net-(U3-PadN10)
- U3 pad N11: (no net) -> Net-(U3-PadN11)
- U3 pad N12: (no net) -> Net-(U3-PadN12)
- U3 pad N13: (no net) -> Net-(U3-PadN13)
- U3 pad N14: (no net) -> Net-(U3-PadN14)
- U3 pad N15: (no net) -> Net-(U3-PadN15)
- U3 pad N16: (no net) -> Net-(U3-PadN16)
- U3 pad N17: (no net) -> Net-(U3-PadN17)
- U3 pad N18: (no net) -> Net-(U3-PadN18)
- U3 pad N19: (no net) -> Net-(U3-PadN19)
- U3 pad N2: (no net) -> Net-(U3-PadN2)
- U3 pad N20: (no net) -> Net-(U3-PadN20)
- U3 pad N21: (no net) -> Net-(U3-PadN21)
- U3 pad N22: (no net) -> Net-(U3-PadN22)
- U3 pad N23: (no net) -> Net-(U3-PadN23)
- U3 pad N3: (no net) -> Net-(U3-PadN3)
- U3 pad N4: (no net) -> Net-(U3-PadN4)
- U3 pad N5: (no net) -> Net-(U3-PadN5)
- U3 pad N6: (no net) -> Net-(U3-PadN6)
- U3 pad N7: (no net) -> Net-(U3-PadN7)
- U3 pad N8: (no net) -> Net-(U3-PadN8)
- U3 pad N9: (no net) -> Net-(U3-PadN9)
- U3 pad S10: (no net) -> Net-(U3-PadS10)
- U3 pad S15: /Interfaces/RS485_OUT_RO -> /Interfaces/RS485_IN_RO
- U3 pad S16: /Interfaces/RS485_OUT_DI -> /Interfaces/RS485_IN_DI
- U3 pad S17: /Interfaces/RS232_OUT_RX -> /Interfaces/RS485_OUT_RO
- U3 pad S18: /Interfaces/RS232_OUT_TX -> /Interfaces/RS485_OUT_DI
- U3 pad S19: (no net) -> Net-(U3-PadS19)
- U3 pad S9: (no net) -> Net-(U3-PadS9)
- U3 pad W10: (no net) -> Net-(U3-PadW10)
- U3 pad W11: (no net) -> Net-(U3-PadW11)
- U3 pad W12: (no net) -> Net-(U3-PadW12)
- U3 pad W13: (no net) -> Net-(U3-PadW13)
- U3 pad W14: (no net) -> Net-(U3-PadW14)
- U3 pad W15: (no net) -> Net-(U3-PadW15)
- U3 pad W16: (no net) -> Net-(U3-PadW16)
- U3 pad W17: (no net) -> Net-(U3-PadW17)
- U3 pad W18: (no net) -> Net-(U3-PadW18)
- U3 pad W19: +3V3 -> /AriaG25Module/ADVREF
- U3 pad W20: /AriaG25Module/3V3_DIV -> /5V_DIV
- U3 pad W21: /AriaG25Module/5V_DIV -> /3V3_DIV
- U3 pad W22: /AriaG25Module/VBUS_DIV -> /VBUS_DIV
- U3 pad W23: /AriaG25Module/VIN_DIV -> /VJACK_DIV
- U3 pad W9: (no net) -> Net-(U3-PadW9)
- U4 pad 11: (no net) -> Net-(U4-Pad11)
- U4 pad 13: (no net) -> Net-(U4-Pad13)
- U4 pad 14: (no net) -> Net-(U4-Pad14)
- U4 pad 15: (no net) -> Net-(U4-Pad15)
- U4 pad 16: (no net) -> Net-(U4-Pad16)
- U4 pad 7: (no net) -> Net-(U4-Pad7)
- U4 pad 8: (no net) -> Net-(U4-Pad8)
- U4 pad 9: (no net) -> Net-(U4-Pad9)
- U5 pad 1: (no net) -> Net-(U5-Pad1)
- U5 pad 14: (no net) -> Net-(U5-Pad14)
- U5 pad 22: (no net) -> Net-(U5-Pad22)
- U5 pad 23: (no net) -> Net-(U5-Pad23)
- U5 pad 29: (no net) -> Net-(U5-Pad29)
- U5 pad 30: (no net) -> Net-(U5-Pad30)
- U5 pad 31: (no net) -> Net-(U5-Pad31)
- U5 pad 32: (no net) -> Net-(U5-Pad32)
- U5 pad 34: (no net) -> Net-(U5-Pad34)
- U5 pad 36: (no net) -> Net-(U5-Pad36)
- U5 pad 37: (no net) -> Net-(U5-Pad37)
- U5 pad 38: (no net) -> Net-(U5-Pad38)
- U5 pad 39: (no net) -> Net-(U5-Pad39)
- U5 pad 40: (no net) -> Net-(U5-Pad40)
- U5 pad 41: (no net) -> Net-(U5-Pad41)
- U5 pad 42: (no net) -> Net-(U5-Pad42)
- U5 pad 43: (no net) -> Net-(U5-Pad43)
- U5 pad 44: (no net) -> Net-(U5-Pad44)
- U5 pad 45: (no net) -> Net-(U5-Pad45)
- U5 pad 46: (no net) -> Net-(U5-Pad46)
- U5 pad 47: (no net) -> Net-(U5-Pad47)
- U5 pad 53: (no net) -> Net-(U5-Pad53)
- U5 pad 54: (no net) -> Net-(U5-Pad54)
- U5 pad 55: (no net) -> Net-(U5-Pad55)
- U5 pad 56: (no net) -> Net-(U5-Pad56)
- U6 pad 2: /Interfaces/RS485_IN_RTS -> /AriaG25Module/PC30
- U6 pad 3: /Interfaces/RS485_IN_RTS -> /AriaG25Module/PC30
- U7 pad 2: /AriaG25Module/PC30 -> /Interfaces/RS485_OUT_RTS
- U7 pad 3: /AriaG25Module/PC30 -> /Interfaces/RS485_OUT_RTS
- W1 pad 1: /VIN -> /VBUS
- W10 pad 1: /Interfaces/RS485_OUT_RO -> /Interfaces/RS485_IN_RO
- W11 pad 1: /Interfaces/RS485_IN_DI -> /Interfaces/RS232_OUT_TX
- W12 pad 1: /Interfaces/RS485_IN_RO -> /Interfaces/RS232_OUT_RX
- W2 pad 1: /VIN -> /VJACK
- W7 pad 1: /Interfaces/RS232_OUT_TX -> /Interfaces/RS485_OUT_DI
- W8 pad 1: /Interfaces/RS232_OUT_RX -> /Interfaces/RS485_OUT_RO
- W9 pad 1: /Interfaces/RS485_OUT_DI -> /Interfaces/RS485_IN_DI
Routing:
- net +3V3: track 0.00 -> 448.1 mm, vias 0 -> 25
- net /VBUS: track 0.00 -> 145.9 mm
- net /Power/VIN: track 0.00 -> 88.9 mm, vias 0 -> 1
- net /Interfaces/RS485_OUT_RTS: track 0.00 -> 86.7 mm, vias 0 -> 2
- net /AriaG25Module/PC30: track 0.00 -> 73.2 mm, vias 0 -> 4
- net +5V: track 0.00 -> 63.6 mm, vias 0 -> 1
- net /Interfaces/USB_ETH_conv/VDD33A: track 0.00 -> 62.7 mm, vias 0 -> 6
- net GND: track 0.00 -> 61.8 mm, vias 0 -> 32
- net /Interfaces/RS485_IN_DI: track 0.00 -> 61.3 mm
- net /AriaG25Module/DRXD: track 0.00 -> 59.6 mm, vias 0 -> 2
- net /Interfaces/RS485_IN_RO: track 0.00 -> 58.6 mm
- net /AriaG25Module/DTXD: track 0.00 -> 58.6 mm, vias 0 -> 2
- net /AriaG25Module/VBAT: track 0.00 -> 53.7 mm, vias 0 -> 2
- net /Interfaces/RS485_OUT_RO: track 0.00 -> 49.1 mm
- net /Interfaces/RS485_OUT_DI: track 0.00 -> 45.1 mm
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